File: KiCad/Snack Machine.sch (KiCad schematic (older format))
At the start: 51 parts, among them J1 AVR-ISP-6, J2 RFID_CONNECTOR, J3 Screw_Terminal_01x08, J4 Screw_Terminal_01x08, J5 Display Serial Header, J6 MDB, U1 MEZD71202A-G, U2 ATmega2560-16AU

Commit message: small tweaks
Parts:
- added J?: MDB, symbol Connector_Generic:Conn_02x03_Top_Bottom
- renumbered J6 to J?
Connections:
- net labels added: RESET_DISPLAY
- wire segments 218 -> 232
- no-connect marks 57 -> 58
Changed lines of the file:
@@
 NoConn ~ 13250 7650
 NoConn ~ 13250 7750
-Text Label 12550 7450 2    50   ~ 0
+Text Label 12350 7450 2    50   ~ 0
 TX_DISPLAY
-Text Label 12550 7550 2    50   ~ 0
+Text Label 12350 7550 2    50   ~ 0
 RX_DISPLAY
 $Comp
@@
 $EndComp
 Text Label 12500 7750 2    50   ~ 0
-~RESET
+RESET_DISPLAY
 $Comp
 L Connector:Conn_01x05_Male J2
@@
 NoConn ~ 9100 8100
 $Sheet
-S 9450 6400 550  300
+S 9450 6400 700  350
 U 5BCD883C
 F0 "USB_Serial" 50
@@
 F2 "RX_USB" I L 9450 6500 50
 F3 "TX_USB" I L 9450 6600 50
+F4 "~RESET" I R 10150 6650 50
 $EndSheet
 Wire Wire Line
@@
 NoConn ~ 9100 8200
 $Comp
-L Connector_Generic:Conn_02x03_Top_Bottom J6
+L Connector_Generic:Conn_02x03_Top_Bottom J?
 U 1 1 5BD02A51
 P 4550 6650
-F 0 "J6" H 4600 6325 50  0000 C CNN
+F 0 "J?" H 4600 6325 50  0000 C CNN
 F 1 "MDB" H 4600 6416 50  0000 C CNN
 F 2 "" H 4550 6650 50  0001 C CNN
@@
 	9100 6000 9800 6000
 Wire Wire Line
-	12100 7550 12750 7550
-Wire Wire Line
-	12100 7450 12750 7450
-Wire Wire Line
-	12100 7750 12750 7750
+	11850 7550 12750 7550
+Wire Wire Line
+	11850 7450 12750 7450
+Wire Wire Line
+	11850 7750 12750 7750
 Wire Wire Line
 	12750 7350 12700 7350
@@
 Connection ~ 6100 7150
 Wire Wire Line
-	4850 6650 5600 6650
+	4850 6650 5050 6650
 Text Notes 5350 7300 0    50   ~ 0
 NOTE: pick resistor vals
@@
 Wire Wire Line
 	4750 9450 5300 9450
-Wire Bus Line
-	10900 2900 10900 3600
-Wire Bus Line
-	9400 2900 9400 3600
-Wire Bus Line
-	10900 3800 10900 4500
-Wire Bus Line
-	10050 4500 10050 5400
 Text Notes 9350 2650 0    50   ~ 0
 CONFLICT? PA0 is AN0
@@
 Text Notes 650  600  0    50   ~ 0
 NOTE: This file is a work-in-progress.  There are many notes which will be removed before release.
+$Comp
+L Connector_Generic:Conn_02x03_Top_Bottom J?
+U 1 1 5BF4B2DB
+P 2650 6650
+F 0 "J?" H 2700 6325 50  0000 C CNN
+F 1 "MDB" H 2700 6416 50  0000 C CNN
+F 2 "" H 2650 6650 50  0001 C CNN
+F 3 "~" H 2650 6650 50  0001 C CNN
+	1    2650 6650
+	1    0    0    1
+$EndComp
+NoConn ~ 2450 6550
+$Comp
+L power:GND #PWR?
+U 1 1 5BF4B2E3
+P 3000 6850
+F 0 "#PWR?" H 3000 6600 50  0001 C CNN
+F 1 "GND" H 3000 6700 50  0000 C CNN
+F 2 "" H 3000 6850 50  0001 C CNN
+F 3 "" H 3000 6850 50  0001 C CNN
+	1    3000 6850
+	1    0    0    -1
+$EndComp
+Wire Wire Line
+	2950 6550 3000 6550
+Wire Wire Line
+	3000 6550 3000 6850
+Wire Wire Line
+	2450 6650 2400 6650
+Wire Wire Line
+	2400 6650 2400 6850
+Wire Wire Line
+	2450 6750 2300 6750
+Wire Wire Line
+	2300 6750 2300 6350
+Wire Wire Line
+	2950 6750 3550 6750
+Wire Wire Line
+	2950 6650 3700 6650
+$Comp
+L power:GND #PWR?
+U 1 1 5BF4B2F1
+P 2400 6850
+F 0 "#PWR?" H 2400 6600 50  0001 C CNN
+F 1 "GND" H 2400 6700 50  0000 C CNN
+F 2 "" H 2400 6850 50  0001 C CNN
+F 3 "" H 2400 6850 50  0001 C CNN
+	1    2400 6850
+	1    0    0    -1
+$EndComp
+$Comp
+L power:+24V #PWR?
+U 1 1 5BF4B2F7
+P 2300 6350
+F 0 "#PWR?" H 2300 6200 50  0001 C CNN
+F 1 "+24V" H 2300 6500 50  0000 C CNN
+F 2 "" H 2300 6350 50  0001 C CNN
+F 3 "" H 2300 6350 50  0001 C CNN
+	1    2300 6350
+	1    0    0    -1
+$EndComp
+Text Label 3150 6750 0    50   ~ 0
+RX_MDB
+Wire Wire Line
+	3700 6650 3700 6050
+Wire Wire Line
+	3700 6050 5050 6050
+Wire Wire Line
+	5050 6050 5050 6650
+Connection ~ 5050 6650
+Wire Wire Line
+	5050 6650 5600 6650
+Text Label 10500 7700 2    50   ~ 0
+RESET_DISPLAY
+Wire Wire Line
+	10700 7700 9800 7700
+Wire Wire Line
+	10150 6650 10550 6650
+Text Label 10250 6650 0    50   ~ 0
+~RESET
+Wire Bus Line
+	10900 2900 10900 3600
+Wire Bus Line
+	9400 2900 9400 3600
+Wire Bus Line
+	10900 3800 10900 4500
+Wire Bus Line
+	10050 4500 10050 5400
 $EndSCHEMATC

Commit message: latest changes, not quite ready to be done, but making commit so we can continue to make layout changes while the schematic is being updated.
Parts:
- removed J2: RFID_CONNECTOR, symbol Connector:Conn_01x05_Male
- removed J? (x2): MDB, symbol Connector_Generic:Conn_02x03_Top_Bottom
- removed TP?: TestPoint, symbol Connector:TestPoint
- added C? (x2): OPEN, symbol Device:C
- added J?: RFID_CONNECTOR, symbol Connector:Conn_01x05_Male
- added J? (x2): MDB, symbol Connector_Generic:Conn_02x03_Top_Bottom
- added R? (x2): 0R, symbol Device:R
- added U?: MEZD71201A-F, symbol Regulator_Linear:uA7805
Connections:
- net labels added: +3.3V, MOTOR_CURRENT
- wire segments 232 -> 248
- no-connect marks 58 -> 47
Other:
- note removed: "ANALOG MOTOR CURRENT?"
- note removed: "CONFLICT? PA0 is AN0"
- note removed: "CONFLICT? PE4-7 are INT4-7"
- moved on the sheet: C?, J3, J4, J5, Q?, R?, Y?

Commit message: Updating annotations for all schematics
Parts:
- gave numbers to parts that had none: 44
- renumbered C1 to C3, C3 to C4, C6 to C5, C7 to C6, C2 to C9, J5 to J11, J1 to J2, R4 to R1, U2 to U3

Commit message: Fixing rescue issue with atmega2560 hopefully
Parts:
- removed U3: ATmega2560-16AU, Package_QFP:TQFP-100_14x14mm_P0.5mm, symbol Snack-Machine-rescue:ATmega2560-16AU-MCU_Microchip_ATmega
- added U?: ATmega2560-16AU, Package_QFP:TQFP-100_14x14mm_P0.5mm, symbol MCU_Microchip_ATmega:ATmega2560-16AU
Changed lines of the file:
@@
 	0    1    1    0
-$EndComp
-$Comp
-L Snack-Machine-rescue:ATmega2560-16AU-MCU_Microchip_ATmega U3
-U 1 1 5BB84FB8
-P 8300 5600
-F 0 "U3" H 8650 2800 50  0000 C CNN
-F 1 "ATmega2560-16AU" H 8750 2700 50  0000 C CNN
-F 2 "Package_QFP:TQFP-100_14x14mm_P0.5mm" H 8300 5600 50  0001 C CIN
-F 3 "http://ww1.microchip.com/downloads/en/DeviceDoc/Atmel-2549-8-bit-AVR-Microcontroller-ATmega640-1280-1281-2560-2561_datasheet.pdf" H 8300 5600 50  0001 C CNN
-	1    8300 5600
-	1    0    0    -1
 $EndComp
 Wire Wire Line
@@
 Wire Wire Line
 	7100 6700 7500 6700
+$Comp
+L MCU_Microchip_ATmega:ATmega2560-16AU U?
+U 1 1 5BFE17CA
+P 8300 5600
+F 0 "U?" H 8300 2614 50  0000 C CNN
+F 1 "ATmega2560-16AU" H 8300 2523 50  0000 C CNN
+F 2 "Package_QFP:TQFP-100_14x14mm_P0.5mm" H 8300 5600 50  0001 C CIN
+F 3 "http://ww1.microchip.com/downloads/en/DeviceDoc/Atmel-2549-8-bit-AVR-Microcontroller-ATmega640-1280-1281-2560-2561_datasheet.pdf" H 8300 5600 50  0001 C CNN
+	1    8300 5600
+	1    0    0    -1
+$EndComp
 $EndSCHEMATC

Commit message: latest changes, mostly test points and annotations
Parts:
- added C15, C16, C17, C18, C19, C20: OPEN, symbol Device:C
- added H1, H2, H3, H4: MountingHole_Pad, symbol Mechanical:MountingHole_Pad
- added J18: Conn_02x15_Counter_Clockwise, symbol Connector_Generic:Conn_02x15_Counter_Clockwise
- added R49, R50, R51, R52, R53, R54: 0R, symbol Device:R
- added TP11, TP12, TP13, TP14, TP15, TP16, TP17, TP18, TP19, TP20, TP21, TP22, TP23, TP24, TP25, TP26, TP27, TP28, TP29, TP30, TP33, TP34, TP35, TP36, TP37, TP38, TP39, TP40, TP41, TP42, TP43, TP44, TP45, TP46, TP47, TP48, TP49, TP50, TP51, TP52, TP55, TP56, TP57, TP58, TP59, TP60, TP61, TP62, TP63, TP64, TP65, TP66, TP67, TP68, TP69, TP70, TP71, TP72, TP73, TP74, TP75, TP76, TP77, TP78, TP79, TP80, TP81, TP82, TP83, TP84, TP85, TP86, TP87, TP88, TP89: TestPoint, symbol Connector:TestPoint
- gave numbers to parts that had none: 1
Connections:
- wire segments 248 -> 377
- no-connect marks 47 -> 7
Other:
- note added: "Input and output caps"
- note removed: "MOUNT HOLES"
- note removed: "NOISE RC"
- moved on the sheet: C11, C12, J10, J11, J3, J4, J5, J6, J7, J8, J9, Q1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

Commit message: Updating components and footprints
Parts:
- C10, C11, C12, C3, C4, C5, C6, C7, C8, C9: footprint (none) -> Capacitor_SMD:C_0603_1608Metric_Pad1.05x0.95mm_HandSolder
- J2: footprint (none) -> Connector_PinHeader_1.00mm:PinHeader_2x03_P1.00mm_Vertical_SMD
- R1, R10, R11, R12, R2, R3, R4, R5, R6, R7, R8, R9: footprint (none) -> Resistor_SMD:R_0603_1608Metric_Pad1.05x0.95mm_HandSolder
- TP1, TP10, TP2, TP6, TP7, TP8, TP9: footprint (none) -> TestPoint:TestPoint_THTPad_D1.0mm_Drill0.5mm
- Y1: footprint (none) -> Crystal:Resonator_SMD_muRata_CSTxExxV-3Pin_3.0x1.1mm_HandSoldering
Changed lines of the file:
@@
 F 0 "J2" H 11350 2000 50  0000 R CNN
 F 1 "AVR-ISP-6" H 11700 1900 50  0000 R CNN
-F 2 "" V 10950 1550 50  0001 C CNN
+F 2 "Connector_PinHeader_1.00mm:PinHeader_2x03_P1.00mm_Vertical_SMD" V 10950 1550 50  0001 C CNN
 F 3 " ~" H 9925 950 50  0001 C CNN
 	1    11200 1500
@@
 F 0 "C4" H 8315 1746 50  0000 L CNN
 F 1 "100nF" H 8315 1655 50  0000 L CNN
-F 2 "" H 8238 1550 50  0001 C CNN
+F 2 "Capacitor_SMD:C_0603_1608Metric_Pad1.05x0.95mm_HandSolder" H 8238 1550 50  0001 C CNN
 F 3 "~" H 8200 1700 50  0001 C CNN
 	1    8200 1700
@@
 F 0 "C5" H 8765 1746 50  0000 L CNN
 F 1 "100nF" H 8765 1655 50  0000 L CNN
-F 2 "" H 8688 1550 50  0001 C CNN
+F 2 "Capacitor_SMD:C_0603_1608Metric_Pad1.05x0.95mm_HandSolder" H 8688 1550 50  0001 C CNN
 F 3 "~" H 8650 1700 50  0001 C CNN
 	1    8650 1700
@@
 F 0 "C6" H 9215 1746 50  0000 L CNN
 F 1 "100nF" H 9215 1655 50  0000 L CNN
-F 2 "" H 9138 1550 50  0001 C CNN
+F 2 "Capacitor_SMD:C_0603_1608Metric_Pad1.05x0.95mm_HandSolder" H 9138 1550 50  0001 C CNN
 F 3 "~" H 9100 1700 50  0001 C CNN
 	1    9100 1700
@@
 F 0 "R1" H 5650 2050 50  0000 C CNN
 F 1 "10K" H 5650 2150 50  0000 C CNN
-F 2 "" V 5730 2100 50  0001 C CNN
+F 2 "Resistor_SMD:R_0603_1608Metric_Pad1.05x0.95mm_HandSolder" V 5730 2100 50  0001 C CNN
 F 3 "~" H 5800 2100 50  0001 C CNN
 	1    5800 2100
@@
 F 0 "C9" H 5915 2646 50  0000 L CNN
 F 1 "22pF" H 5915 2555 50  0000 L CNN
-F 2 "" H 5838 2450 50  0001 C CNN
+F 2 "Capacitor_SMD:C_0603_1608Metric_Pad1.05x0.95mm_HandSolder" H 5838 2450 50  0001 C CNN
 F 3 "~" H 5800 2600 50  0001 C CNN
 	1    5800 2600
@@
 F 0 "R3" H 5170 4046 50  0000 L CNN
 F 1 "1M" H 5170 3955 50  0000 L CNN
-F 2 "" V 5030 4000 50  0001 C CNN
+F 2 "Resistor_SMD:R_0603_1608Metric_Pad1.05x0.95mm_HandSolder" V 5030 4000 50  0001 C CNN
 F 3 "~" H 5100 4000 50  0001 C CNN
 	1    5100 4000
@@
 F 0 "C8" H 10115 1746 50  0000 L CNN
 F 1 "1uF" H 10115 1655 50  0000 L CNN
-F 2 "" H 10038 1550 50  0001 C CNN
+F 2 "Capacitor_SMD:C_0603_1608Metric_Pad1.05x0.95mm_HandSolder" H 10038 1550 50  0001 C CNN
 F 3 "~" H 10000 1700 50  0001 C CNN
 	1    10000 1700
@@
 F 0 "Y1" V 4646 4131 50  0000 L CNN
 F 1 "16MHz" V 4555 4131 50  0000 L CNN
-F 2 "" H 4600 4000 50  0001 C CNN
+F 2 "Crystal:Resonator_SMD_muRata_CSTxExxV-3Pin_3.0x1.1mm_HandSoldering" H 4600 4000 50  0001 C CNN
 F 3 "~" H 4600 4000 50  0001 C CNN
 F 4 "Murata" H 4600 4000 50  0001 C CNN "Manufacturer"
@@
 F 0 "C10" H 6865 3846 50  0000 L CNN
 F 1 "100nF" H 6865 3755 50  0000 L CNN
-F 2 "" H 6788 3650 50  0001 C CNN
+F 2 "Capacitor_SMD:C_0603_1608Metric_Pad1.05x0.95mm_HandSolder" H 6788 3650 50  0001 C CNN
 F 3 "~" H 6750 3800 50  0001 C CNN
 	1    6750 3800
@@
 F 0 "C7" H 9665 1746 50  0000 L CNN
 F 1 "100nF" H 9665 1655 50  0000 L CNN
-F 2 "" H 9588 1550 50  0001 C CNN
+F 2 "Capacitor_SMD:C_0603_1608Metric_Pad1.05x0.95mm_HandSolder" H 9588 1550 50  0001 C CNN
 F 3 "~" H 9550 1700 50  0001 C CNN
 	1    9550 1700
@@
 F 0 "R10" H 14000 6900 50  0000 C CNN
 F 1 "10K" H 14000 6800 50  0000 C CNN
-F 2 "" V 13780 6850 50  0001 C CNN
+F 2 "Resistor_SMD:R_0603_1608Metric_Pad1.05x0.95mm_HandSolder" V 13780 6850 50  0001 C CNN
 F 3 "~" H 13850 6850 50  0001 C CNN
 	1    13850 6850
@@
 F 0 "R11" H 14350 6900 50  0000 C CNN
 F 1 "10K" H 14350 6800 50  0000 C CNN
-F 2 "" V 14130 6850 50  0001 C CNN
+F 2 "Resistor_SMD:R_0603_1608Metric_Pad1.05x0.95mm_HandSolder" V 14130 6850 50  0001 C CNN
 F 3 "~" H 14200 6850 50  0001 C CNN
 	1    14200 6850
@@
 F 0 "R8" H 4150 6650 50  0000 C CNN
 F 1 "10K" H 4150 6750 50  0000 C CNN
-F 2 "" V 4230 6700 50  0001 C CNN
+F 2 "Resistor_SMD:R_0603_1608Metric_Pad1.05x0.95mm_HandSolder" V 4230 6700 50  0001 C CNN
 F 3 "~" H 4300 6700 50  0001 C CNN
 	1    4300 6700
@@
 F 0 "R12" V 4500 7000 50  0000 C CNN
 F 1 "10K" V 4400 7000 50  0000 C CNN
-F 2 "" V 4530 7000 50  0001 C CNN
+F 2 "Resistor_SMD:R_0603_1608Metric_Pad1.05x0.95mm_HandSolder" V 4530 7000 50  0001 C CNN
 F 3 "~" H 4600 7000 50  0001 C CNN
 	1    4600 7000
@@
 F 0 "TP2" V 9150 4250 50  0000 L CNN
 F 1 "TestPoint" V 9150 4500 50  0000 L CNN
-F 2 "" H 9400 4300 50  0001 C CNN
+F 2 "TestPoint:TestPoint_THTPad_D1.0mm_Drill0.5mm" H 9400 4300 50  0001 C CNN
 F 3 "~" H 9400 4300 50  0001 C CNN
 	1    9200 4300
@@
 F 0 "TP1" V 9150 3850 50  0000 L CNN
 F 1 "TestPoint" V 9150 4100 50  0000 L CNN
-F 2 "" H 9400 3900 50  0001 C CNN
+F 2 "TestPoint:TestPoint_THTPad_D1.0mm_Drill0.5mm" H 9400 3900 50  0001 C CNN
 F 3 "~" H 9400 3900 50  0001 C CNN
 	1    9200 3900
@@
 F 0 "R5" V 5800 5750 50  0000 C CNN
 F 1 "0R" V 5800 5350 50  0000 C CNN
-F 2 "" V 5680 5550 50  0001 C CNN
+F 2 "Resistor_SMD:R_0603_1608Metric_Pad1.05x0.95mm_HandSolder" V 5680 5550 50  0001 C CNN
 F 3 "~" H 5750 5550 50  0001 C CNN
 	1    5750 5550
@@
 F 0 "R6" V 5800 5850 50  0000 C CNN
 F 1 "0R" V 5800 5450 50  0000 C CNN
-F 2 "" V 5680 5650 50  0001 C CNN
+F 2 "Resistor_SMD:R_0603_1608Metric_Pad1.05x0.95mm_HandSolder" V 5680 5650 50  0001 C CNN
 F 3 "~" H 5750 5650 50  0001 C CNN
 	1    5750 5650
@@
 F 0 "C3" H 7865 1746 50  0000 L CNN
 F 1 "100nF" H 7865 1655 50  0000 L CNN
-F 2 "" H 7788 1550 50  0001 C CNN
+F 2 "Capacitor_SMD:C_0603_1608Metric_Pad1.05x0.95mm_HandSolder" H 7788 1550 50  0001 C CNN
 F 3 "~" H 7750 1700 50  0001 C CNN
 	1    7750 1700
@@
 F 0 "R4" H 3450 5150 50  0000 C CNN
 F 1 "10K" H 3450 5250 50  0000 C CNN
-F 2 "" V 3530 5200 50  0001 C CNN
+F 2 "Resistor_SMD:R_0603_1608Metric_Pad1.05x0.95mm_HandSolder" V 3530 5200 50  0001 C CNN
 F 3 "~" H 3600 5200 50  0001 C CNN
 	1    3600 5200
@@
 F 0 "R2" H 5050 3000 50  0000 C CNN
 F 1 "1K" H 5050 3100 50  0000 C CNN
-F 2 "" V 5130 3050 50  0001 C CNN
+F 2 "Resistor_SMD:R_0603_1608Metric_Pad1.05x0.95mm_HandSolder" V 5130 3050 50  0001 C CNN
 F 3 "~" H 5200 3050 50  0001 C CNN
 	1    5200 3050
@@
 F 0 "TP7" V 5250 9200 50  0000 L CNN
 F 1 "TestPoint" V 5250 9450 50  0000 L CNN
-F 2 "" H 5500 9250 50  0001 C CNN
+F 2 "TestPoint:TestPoint_THTPad_D1.0mm_Drill0.5mm" H 5500 9250 50  0001 C CNN
 F 3 "~" H 5500 9250 50  0001 C CNN
 	1    5300 9250
@@
 F 0 "TP8" V 5250 9300 50  0000 L CNN
 F 1 "TestPoint" V 5250 9550 50  0000 L CNN
-F 2 "" H 5500 9350 50  0001 C CNN
+F 2 "TestPoint:TestPoint_THTPad_D1.0mm_Drill0.5mm" H 5500 9350 50  0001 C CNN
 F 3 "~" H 5500 9350 50  0001 C CNN
 	1    5300 9350
@@
 F 0 "TP9" V 5250 9400 50  0000 L CNN
 F 1 "TestPoint" V 5250 9650 50  0000 L CNN
-F 2 "" H 5500 9450 50  0001 C CNN
+F 2 "TestPoint:TestPoint_THTPad_D1.0mm_Drill0.5mm" H 5500 9450 50  0001 C CNN
 F 3 "~" H 5500 9450 50  0001 C CNN
 	1    5300 9450
@@
 F 0 "TP6" V 3550 9200 50  0000 L CNN
 F 1 "TestPoint" V 3550 9450 50  0000 L CNN
-F 2 "" H 3800 9250 50  0001 C CNN
+F 2 "TestPoint:TestPoint_THTPad_D1.0mm_Drill0.5mm" H 3800 9250 50  0001 C CNN
 F 3 "~" H 3800 9250 50  0001 C CNN
 	1    3600 9250
@@
 F 0 "TP10" V 3550 9500 50  0000 L CNN
 F 1 "TestPoint" V 3550 9750 50  0000 L CNN
-F 2 "" H 3800 9550 50  0001 C CNN
+F 2 "TestPoint:TestPoint_THTPad_D1.0mm_Drill0.5mm" H 3800 9550 50  0001 C CNN
 F 3 "~" H 3800 9550 50  0001 C CNN
 	1    3600 9550
@@
 F 0 "C12" H 6465 6996 50  0000 L CNN
 F 1 "OPEN" H 6465 6905 50  0000 L CNN
-F 2 "" H 6388 6800 50  0001 C CNN
+F 2 "Capacitor_SMD:C_0603_1608Metric_Pad1.05x0.95mm_HandSolder" H 6388 6800 50  0001 C CNN
 F 3 "~" H 6350 6950 50  0001 C CNN
 	1    6350 6950
@@
 F 0 "C11" H 5800 7000 50  0000 L CNN
 F 1 "OPEN" H 5700 6900 50  0000 L CNN
-F 2 "" H 6088 6800 50  0001 C CNN
+F 2 "Capacitor_SMD:C_0603_1608Metric_Pad1.05x0.95mm_HandSolder" H 6088 6800 50  0001 C CNN
 F 3 "~" H 6050 6950 50  0001 C CNN
 	1    6050 6950
@@
 F 0 "R7" V 5800 6800 50  0000 C CNN
 F 1 "0R" V 5800 6400 50  0000 C CNN
-F 2 "" V 5680 6600 50  0001 C CNN
+F 2 "Resistor_SMD:R_0603_1608Metric_Pad1.05x0.95mm_HandSolder" V 5680 6600 50  0001 C CNN
 F 3 "~" H 5750 6600 50  0001 C CNN
 	1    5750 6600
@@
 F 0 "R9" V 5800 6900 50  0000 C CNN
 F 1 "0R" V 5800 6500 50  0000 C CNN
-F 2 "" V 5680 6700 50  0001 C CNN
+F 2 "Resistor_SMD:R_0603_1608Metric_Pad1.05x0.95mm_HandSolder" V 5680 6700 50  0001 C CNN
 F 3 "~" H 5750 6700 50  0001 C CNN
 	1    5750 6700
@@
 U 1 1 5BFE17CA
 P 8300 5600
-F 0 "U3" H 8550 2800 50  0000 C CNN
-F 1 "ATmega2560-16AU" H 8850 2700 50  0000 C CNN
+F 0 "U3" H 8900 2700 50  0000 C CNN
+F 1 "ATmega2560-16AU" H 8750 2800 50  0000 C CNN
 F 2 "Package_QFP:TQFP-100_14x14mm_P0.5mm" H 8300 5600 50  0001 C CIN
 F 3 "http://ww1.microchip.com/downloads/en/DeviceDoc/Atmel-2549-8-bit-AVR-Microcontroller-ATmega640-1280-1281-2560-2561_datasheet.pdf" H 8300 5600 50  0001 C CNN

Commit message: changed all mosfets
Parts:
- Q1: value P-CH 10V 200mA -> P-CH 30V 3.8A; symbol Transistor_FET:BSS83P -> Device:Q_PMOS_GSD; Part Number DMG2305UX-13 -> DMP3099L-7
Changed lines of the file:
@@
 	11100 1900 11100 1950
 $Comp
-L Transistor_FET:BSS83P Q1
+L Device:Q_PMOS_GSD Q1
 U 1 1 5C41527C
 P 4000 6600
 F 0 "Q1" V 4343 6600 50  0000 C CNN
-F 1 "P-CH 10V 200mA" V 4252 6600 50  0000 C CNN
+F 1 "P-CH 30V 3.8A" V 4252 6600 50  0000 C CNN
 F 2 "TO_SOT_Packages_SMD:SOT-23_Handsoldering" H 4200 6525 50  0001 L CIN
 F 3 "~" H 4000 6600 50  0001 L CNN
 F 4 "Diodes Incorporated" H 4000 6600 50  0001 C CNN "Manufacturer"
-F 5 "DMG2305UX-13" H 4000 6600 50  0001 C CNN "Part Number"
+F 5 "DMP3099L-7" H 4000 6600 50  0001 C CNN "Part Number"
 	1    4000 6600
 	0    -1   -1   0
@@
 U 1 1 5BFE17CA
 P 8300 5600
-F 0 "U3" H 8900 2700 50  0000 C CNN
-F 1 "ATmega2560-16AU" H 8750 2800 50  0000 C CNN
+F 0 "U3" H 8800 2800 50  0000 C CNN
+F 1 "ATmega2560-16AU" H 8950 2700 50  0000 C CNN
 F 2 "Package_QFP:TQFP-100_14x14mm_P0.5mm" H 8300 5600 50  0001 C CIN
 F 3 "http://ww1.microchip.com/downloads/en/DeviceDoc/Atmel-2549-8-bit-AVR-Microcontroller-ATmega640-1280-1281-2560-2561_datasheet.pdf" H 8300 5600 50  0001 C CNN
