File: KiCad/Ethernet.sch (KiCad schematic (older format))
At the start: 35 parts

Commit message: Annotating schematic
Parts:
- C31, C32: renamed from C?; value C -> 22pF; footprint (none) -> Capacitor_SMD:C_0603_1608Metric_Pad1.05x0.95mm_HandSolder
- C33, C34, C35, C36, C37, C38, C39, C40, C41, C42, C43, C44: renamed from C?; footprint (none) -> Capacitor_SMD:C_0603_1608Metric_Pad1.05x0.95mm_HandSolder
- gave numbers to parts that had none: 21
Connections:
- wire segments 129 -> 131
Other:
- moved on the sheet: C31, C32

Commit message: Adding more footprints
Parts:
- R64, R65, R66, R67, R68, R69, R70, R71, R72, R73, R74, R75, R76, R77, R78: footprint (none) -> Resistor_SMD:R_0603_1608Metric_Pad1.05x0.95mm_HandSolder
- U7: footprint (none) -> Package_TO_SOT_SMD:SOT-23-5_HandSoldering
- U8: footprint (none) -> Package_QFP:TQFP-48_7x7mm_P0.5mm
Changed lines of the file:
@@
 EESchema Schematic File Version 4
+LIBS:Snack Machine-cache
 EELAYER 26 0
 EELAYER END
@@
 F 0 "U8" H 4250 2450 50  0000 L CNN
 F 1 "W5500" H 2450 2450 50  0000 L CNN
-F 2 "" H 3400 3450 50  0001 C CNN
+F 2 "Package_QFP:TQFP-48_7x7mm_P0.5mm" H 3400 3450 50  0001 C CNN
 F 3 "" H 3400 3450 50  0001 C CNN
 	1    3400 3450
@@
 F 0 "R72" H 3870 1996 50  0000 L CNN
 F 1 "10k" H 3870 1905 50  0000 L CNN
-F 2 "" V 3730 1950 50  0001 C CNN
+F 2 "Resistor_SMD:R_0603_1608Metric_Pad1.05x0.95mm_HandSolder" V 3730 1950 50  0001 C CNN
 F 3 "~" H 3800 1950 50  0001 C CNN
 	1    3800 1950
@@
 F 0 "R70" H 3370 1996 50  0000 L CNN
 F 1 "10k" H 3370 1905 50  0000 L CNN
-F 2 "" V 3230 1950 50  0001 C CNN
+F 2 "Resistor_SMD:R_0603_1608Metric_Pad1.05x0.95mm_HandSolder" V 3230 1950 50  0001 C CNN
 F 3 "~" H 3300 1950 50  0001 C CNN
 	1    3300 1950
@@
 F 0 "R71" H 3620 1996 50  0000 L CNN
 F 1 "10k" H 3620 1905 50  0000 L CNN
-F 2 "" V 3480 1950 50  0001 C CNN
+F 2 "Resistor_SMD:R_0603_1608Metric_Pad1.05x0.95mm_HandSolder" V 3480 1950 50  0001 C CNN
 F 3 "~" H 3550 1950 50  0001 C CNN
 	1    3550 1950
@@
 F 0 "R69" H 2920 1996 50  0000 L CNN
 F 1 "10k" H 2920 1905 50  0000 L CNN
-F 2 "" V 2780 1950 50  0001 C CNN
+F 2 "Resistor_SMD:R_0603_1608Metric_Pad1.05x0.95mm_HandSolder" V 2780 1950 50  0001 C CNN
 F 3 "~" H 2850 1950 50  0001 C CNN
 	1    2850 1950
@@
 F 0 "R67" H 2020 2746 50  0000 L CNN
 F 1 "10k" H 2020 2655 50  0000 L CNN
-F 2 "" V 1880 2700 50  0001 C CNN
+F 2 "Resistor_SMD:R_0603_1608Metric_Pad1.05x0.95mm_HandSolder" V 1880 2700 50  0001 C CNN
 F 3 "~" H 1950 2700 50  0001 C CNN
 	1    1950 2700
@@
 F 0 "R64" V 1200 3500 50  0000 C CNN
 F 1 "1M" V 1100 3500 50  0000 C CNN
-F 2 "" V 1030 3500 50  0001 C CNN
+F 2 "Resistor_SMD:R_0603_1608Metric_Pad1.05x0.95mm_HandSolder" V 1030 3500 50  0001 C CNN
 F 3 "~" H 1100 3500 50  0001 C CNN
 	1    1100 3500
@@
 F 0 "R68" H 2220 4296 50  0000 L CNN
 F 1 "470" H 2220 4205 50  0000 L CNN
-F 2 "" V 2080 4250 50  0001 C CNN
+F 2 "Resistor_SMD:R_0603_1608Metric_Pad1.05x0.95mm_HandSolder" V 2080 4250 50  0001 C CNN
 F 3 "~" H 2150 4250 50  0001 C CNN
 	1    2150 4250
@@
 F 0 "R66" H 1920 4296 50  0000 L CNN
 F 1 "470" H 1920 4205 50  0000 L CNN
-F 2 "" V 1780 4250 50  0001 C CNN
+F 2 "Resistor_SMD:R_0603_1608Metric_Pad1.05x0.95mm_HandSolder" V 1780 4250 50  0001 C CNN
 F 3 "~" H 1850 4250 50  0001 C CNN
 	1    1850 4250
@@
 F 0 "R73" V 5043 3800 50  0000 C CNN
 F 1 "R" V 5134 3800 50  0000 C CNN
-F 2 "" V 5180 3800 50  0001 C CNN
+F 2 "Resistor_SMD:R_0603_1608Metric_Pad1.05x0.95mm_HandSolder" V 5180 3800 50  0001 C CNN
 F 3 "~" H 5250 3800 50  0001 C CNN
 	1    5250 3800
@@
 F 0 "R65" H 1270 3196 50  0000 L CNN
 F 1 "10K" H 1270 3105 50  0000 L CNN
-F 2 "" V 1130 3150 50  0001 C CNN
+F 2 "Resistor_SMD:R_0603_1608Metric_Pad1.05x0.95mm_HandSolder" V 1130 3150 50  0001 C CNN
 F 3 "~" H 1200 3150 50  0001 C CNN
 	1    1200 3150
@@
 F 0 "U7" H 1800 7365 50  0000 C CNN
 F 1 "74AHC1G125" H 1800 7274 50  0000 C CNN
-F 2 "" H 1800 7000 50  0001 C CNN
+F 2 "Package_TO_SOT_SMD:SOT-23-5_HandSoldering" H 1800 7000 50  0001 C CNN
 F 3 "" H 1800 7000 50  0001 C CNN
 	1    1800 7000
@@
 F 0 "R77" H 8770 1296 50  0000 L CNN
 F 1 "49.9" H 8770 1205 50  0000 L CNN
-F 2 "" V 8630 1250 50  0001 C CNN
+F 2 "Resistor_SMD:R_0603_1608Metric_Pad1.05x0.95mm_HandSolder" V 8630 1250 50  0001 C CNN
 F 3 "~" H 8700 1250 50  0001 C CNN
 	1    8700 1250
@@
 F 0 "R78" H 9070 1296 50  0000 L CNN
 F 1 "10" H 9070 1205 50  0000 L CNN
-F 2 "" V 8930 1250 50  0001 C CNN
+F 2 "Resistor_SMD:R_0603_1608Metric_Pad1.05x0.95mm_HandSolder" V 8930 1250 50  0001 C CNN
 F 3 "~" H 9000 1250 50  0001 C CNN
 	1    9000 1250
@@
 F 0 "R75" H 8470 1296 50  0000 L CNN
 F 1 "49.9" H 8470 1205 50  0000 L CNN
-F 2 "" V 8330 1250 50  0001 C CNN
+F 2 "Resistor_SMD:R_0603_1608Metric_Pad1.05x0.95mm_HandSolder" V 8330 1250 50  0001 C CNN
 F 3 "~" H 8400 1250 50  0001 C CNN
 	1    8400 1250
@@
 F 0 "R76" H 8670 2996 50  0000 L CNN
 F 1 "49.9" H 8670 2905 50  0000 L CNN
-F 2 "" V 8530 2950 50  0001 C CNN
+F 2 "Resistor_SMD:R_0603_1608Metric_Pad1.05x0.95mm_HandSolder" V 8530 2950 50  0001 C CNN
 F 3 "~" H 8600 2950 50  0001 C CNN
 	1    8600 2950
@@
 F 0 "R74" H 8370 2996 50  0000 L CNN
 F 1 "49.9" H 8370 2905 50  0000 L CNN
-F 2 "" V 8230 2950 50  0001 C CNN
+F 2 "Resistor_SMD:R_0603_1608Metric_Pad1.05x0.95mm_HandSolder" V 8230 2950 50  0001 C CNN
 F 3 "~" H 8300 2950 50  0001 C CNN
 	1    8300 2950

Commit message: Added Ethernet jack
Parts:
- U9: footprint (none) -> Snack Machine:RB1-125BAG1A
Changed lines of the file:
@@
 F 0 "U9" H 10477 2296 50  0000 L CNN
 F 1 "RB1-125BAG1A" H 10477 2205 50  0000 L CNN
-F 2 "" H 10050 2250 50  0001 C CNN
+F 2 "Snack Machine:RB1-125BAG1A" H 10050 2250 50  0001 C CNN
 F 3 "" H 10050 2250 50  0001 C CNN
 	1    10050 2250

Commit message: Pushing up current changes
Connections:
- wire segments 131 -> 135
Changed lines of the file:
@@
 Wire Wire Line
 	3750 5000 3750 4600
-$Comp
-L power:GND #PWR0124
-U 1 1 5C087172
-P 3850 4700
-F 0 "#PWR0124" H 3850 4450 50  0001 C CNN
-F 1 "GND" H 3855 4527 50  0000 C CNN
-F 2 "" H 3850 4700 50  0001 C CNN
-F 3 "" H 3850 4700 50  0001 C CNN
-	1    3850 4700
-	1    0    0    -1
-$EndComp
-$Comp
-L power:GND #PWR0122
-U 1 1 5C087207
-P 3650 4700
-F 0 "#PWR0122" H 3650 4450 50  0001 C CNN
-F 1 "GND" H 3655 4527 50  0000 C CNN
-F 2 "" H 3650 4700 50  0001 C CNN
-F 3 "" H 3650 4700 50  0001 C CNN
-	1    3650 4700
-	1    0    0    -1
-$EndComp
-$Comp
-L power:GND #PWR0120
-U 1 1 5C08729C
-P 3350 4700
-F 0 "#PWR0120" H 3350 4450 50  0001 C CNN
-F 1 "GND" H 3355 4527 50  0000 C CNN
-F 2 "" H 3350 4700 50  0001 C CNN
-F 3 "" H 3350 4700 50  0001 C CNN
-	1    3350 4700
-	1    0    0    -1
-$EndComp
 Wire Wire Line
 	3350 4700 3350 4600
@@
 Wire Wire Line
 	1250 4350 1300 4350
+Wire Wire Line
+	3350 4700 3650 4700
+Wire Wire Line
+	3650 4700 3850 4700
+Connection ~ 3650 4700
+Wire Wire Line
+	3850 4700 3850 4800
+Connection ~ 3850 4700
+Text Label 4050 4800 2    50   ~ 0
+AGND
+Wire Wire Line
+	4050 4800 3850 4800
 $EndSCHEMATC
