File: KiCad/Ethernet.sch (KiCad schematic (older format))
At the start: 35 parts, among them U7 74AHC1G125, U8 W5500, U9 RB1-125BAG1A, Y3 Crystal

Commit message: added parts for Y3, FB2, FB3, F1
Parts:
- FB2, FB3: Manufacturer (none) -> Murata; Part Number (none) -> BLM21PG221SN1D
- Y3: Manufacturer (none) -> EPSON; Part Number (none) -> TSX-3225 25.0000MF10P-C0
Changed lines of the file:
@@
 EESchema Schematic File Version 4
-LIBS:Snack Machine-cache
 EELAYER 26 0
 EELAYER END
@@
 F 2 "" H 1100 4150 50  0001 C CNN
 F 3 "~" H 1100 4150 50  0001 C CNN
+F 4 "EPSON" H 1100 4150 50  0001 C CNN "Manufacturer"
+F 5 "TSX-3225 25.0000MF10P-C0" H 1100 4150 50  0001 C CNN "Part Number"
 	1    1100 4150
 	1    0    0    -1
@@
 F 2 "" V 4880 5900 50  0001 C CNN
 F 3 "~" H 4950 5900 50  0001 C CNN
+F 4 "Murata" V 4950 5900 50  0001 C CNN "Manufacturer"
+F 5 "BLM21PG221SN1D" V 4950 5900 50  0001 C CNN "Part Number"
 	1    4950 5900
 	0    1    1    0
@@
 F 2 "" V 4880 6400 50  0001 C CNN
 F 3 "~" H 4950 6400 50  0001 C CNN
+F 4 "Murata" V 4950 6400 50  0001 C CNN "Manufacturer"
+F 5 "BLM21PG221SN1D" V 4950 6400 50  0001 C CNN "Part Number"
 	1    4950 6400
 	0    1    1    0
