File: KiCad/Ethernet.sch (KiCad schematic (older format))
At the start: 35 parts, among them U7 74AHC1G125, U8 W5500, U9 RB1-125BAG1A, Y3 Crystal

Commit message: fixed schematic rules check, generated netlist
Connections:
- wire segments 135 -> 138
Changed lines of the file:
@@
 Connection ~ 1700 5450
 Wire Wire Line
-	1250 3500 1250 4350
-Wire Wire Line
-	950  3400 950  4350
+	1250 3500 1250 4150
+Wire Wire Line
+	950  3400 950  3500
 $Comp
 L Device:R R68
@@
 Wire Wire Line
 	4050 4800 3850 4800
+Connection ~ 1250 3500
+Connection ~ 950  3500
+Wire Wire Line
+	950  3500 950  4150
+Connection ~ 950  4150
+Wire Wire Line
+	950  4150 950  4350
+Connection ~ 1250 4150
+Wire Wire Line
+	1250 4150 1250 4350
 $EndSCHEMATC

Commit message: tweaked ethernet
Parts:
- added C45: 10nF, Capacitor_SMD:C_0603_1608Metric_Pad1.05x0.95mm_HandSolder, symbol Device:C
- C33: value 10u -> 10uF
- C34: value 0.1 -> 0.1uF
- R73: value R -> 12.1k
- Y3: value Crystal -> 25MHz
Connections:
- net labels added: TX+, TX-
- wire segments 138 -> 149
Other:
- moved on the sheet: C33
Changed lines of the file:
@@
 	2100 3000 2250 3000
 Wire Wire Line
-	2100 3100 2250 3100
+	1500 3100 2250 3100
 Wire Wire Line
 	2250 3200 2100 3200
@@
 P 1100 4150
 F 0 "Y3" H 1100 4418 50  0000 C CNN
-F 1 "Crystal" H 1100 4327 50  0000 C CNN
+F 1 "25MHz" H 1100 4327 50  0000 C CNN
 F 2 "" H 1100 4150 50  0001 C CNN
 F 3 "~" H 1100 4150 50  0001 C CNN
@@
 P 1700 5650
 F 0 "C34" H 1815 5696 50  0000 L CNN
-F 1 "0.1" H 1815 5605 50  0000 L CNN
+F 1 "0.1uF" H 1815 5605 50  0000 L CNN
 F 2 "Capacitor_SMD:C_0603_1608Metric_Pad1.05x0.95mm_HandSolder" H 1738 5500 50  0001 C CNN
 F 3 "~" H 1700 5650 50  0001 C CNN
@@
 L Device:C C33
 U 1 1 5C07A1CE
-P 1350 5650
-F 0 "C33" H 1465 5696 50  0000 L CNN
-F 1 "10u" H 1465 5605 50  0000 L CNN
-F 2 "Capacitor_SMD:C_0603_1608Metric_Pad1.05x0.95mm_HandSolder" H 1388 5500 50  0001 C CNN
-F 3 "~" H 1350 5650 50  0001 C CNN
-	1    1350 5650
+P 1300 5650
+F 0 "C33" H 1415 5696 50  0000 L CNN
+F 1 "10uF" H 1415 5605 50  0000 L CNN
+F 2 "Capacitor_SMD:C_0603_1608Metric_Pad1.05x0.95mm_HandSolder" H 1338 5500 50  0001 C CNN
+F 3 "~" H 1300 5650 50  0001 C CNN
+	1    1300 5650
 	1    0    0    -1
 $EndComp
@@
 L power:+3.3V #PWR0111
 U 1 1 5C07A266
-P 1350 5400
-F 0 "#PWR0111" H 1350 5250 50  0001 C CNN
-F 1 "+3.3V" H 1365 5573 50  0000 C CNN
-F 2 "" H 1350 5400 50  0001 C CNN
-F 3 "" H 1350 5400 50  0001 C CNN
-	1    1350 5400
+P 1300 5400
+F 0 "#PWR0111" H 1300 5250 50  0001 C CNN
+F 1 "+3.3V" H 1315 5573 50  0000 C CNN
+F 2 "" H 1300 5400 50  0001 C CNN
+F 3 "" H 1300 5400 50  0001 C CNN
+	1    1300 5400
 	1    0    0    -1
 $EndComp
@@
 L power:GND #PWR0112
 U 1 1 5C07A929
-P 1350 5900
-F 0 "#PWR0112" H 1350 5650 50  0001 C CNN
-F 1 "GND" H 1355 5727 50  0000 C CNN
-F 2 "" H 1350 5900 50  0001 C CNN
-F 3 "" H 1350 5900 50  0001 C CNN
-	1    1350 5900
-	1    0    0    -1
-$EndComp
-Wire Wire Line
-	1350 5900 1350 5800
+P 1300 5900
+F 0 "#PWR0112" H 1300 5650 50  0001 C CNN
+F 1 "GND" H 1305 5727 50  0000 C CNN
+F 2 "" H 1300 5900 50  0001 C CNN
+F 3 "" H 1300 5900 50  0001 C CNN
+	1    1300 5900
+	1    0    0    -1
+$EndComp
+Wire Wire Line
+	1300 5900 1300 5800
 $Comp
 L power:GND #PWR0114
@@
 	1700 5900 1700 5800
 Wire Wire Line
-	1700 5450 1700 5500
-Wire Wire Line
-	1700 5450 1700 3700
-Wire Wire Line
 	1700 3700 2250 3700
-Connection ~ 1700 5450
 Wire Wire Line
 	1250 3500 1250 4150
@@
 GREENLED
 Wire Wire Line
-	1350 5450 1350 5400
-Wire Wire Line
-	1350 5450 1700 5450
-Wire Wire Line
-	1350 5450 1350 5500
-Connection ~ 1350 5450
+	1300 5450 1300 5400
+Wire Wire Line
+	1300 5450 1700 5450
+Wire Wire Line
+	1300 5450 1300 5500
+Connection ~ 1300 5450
 $Comp
 L power:GND #PWR0118
@@
 	3550 5000 3150 5000
 Wire Wire Line
-	4650 3700 4550 3700
-Wire Wire Line
-	4550 3100 4650 3100
+	4900 3700 4550 3700
+Wire Wire Line
+	4550 3100 4900 3100
 Wire Wire Line
 	4550 3900 5000 3900
@@
 P 5250 3800
 F 0 "R73" V 5043 3800 50  0000 C CNN
-F 1 "R" V 5134 3800 50  0000 C CNN
+F 1 "12.1k" V 5134 3800 50  0000 C CNN
 F 2 "Resistor_SMD:R_0603_1608Metric_Pad1.05x0.95mm_HandSolder" V 5180 3800 50  0001 C CNN
 F 3 "~" H 5250 3800 50  0001 C CNN
@@
 	5400 6400 5100 6400
 $Comp
-L Device:R R65
-U 1 1 5C0B07F0
-P 1200 3150
-F 0 "R65" H 1270 3196 50  0000 L CNN
-F 1 "10K" H 1270 3105 50  0000 L CNN
-F 2 "Resistor_SMD:R_0603_1608Metric_Pad1.05x0.95mm_HandSolder" V 1130 3150 50  0001 C CNN
-F 3 "~" H 1200 3150 50  0001 C CNN
-	1    1200 3150
-	1    0    0    -1
-$EndComp
-$Comp
 L power:+3.3V #PWR0109
 U 1 1 5C0B3FAA
@@
 Text Label 2100 3100 2    50   ~ 0
 MISO_TRISTATE
-Wire Wire Line
-	1200 3000 1200 2900
-Wire Wire Line
-	1200 3300 2250 3300
-Wire Wire Line
-	1200 3300 900  3300
-Connection ~ 1200 3300
 Text Label 1200 7000 2    50   ~ 0
 MISO_TRISTATE
 Wire Wire Line
-	1200 7000 1300 7000
+	600  7000 1300 7000
 Text HLabel 1200 6900 0    50   Input ~ 0
 CS
@@
 RX+
 Wire Wire Line
-	8100 2500 8300 2500
+	8050 2500 8300 2500
 Wire Wire Line
 	8300 2800 8300 2500
@@
 RX-
 Wire Wire Line
-	8100 2700 8600 2700
+	8050 2700 8600 2700
 Wire Wire Line
 	8600 2800 8600 2700
@@
 Wire Wire Line
 	1250 4150 1250 4350
+Wire Wire Line
+	4550 2900 4900 2900
+Wire Wire Line
+	4550 3000 4900 3000
+Text Label 4650 2900 0    50   ~ 0
+TX-
+Text Label 4650 3000 0    50   ~ 0
+TX+
+Wire Wire Line
+	8700 1500 8100 1500
+Connection ~ 8700 1500
+Wire Wire Line
+	8400 1700 8100 1700
+Connection ~ 8400 1700
+Text Label 8150 1500 0    50   ~ 0
+TX+
+Text Label 8150 1700 0    50   ~ 0
+TX-
+Wire Wire Line
+	4550 3300 4900 3300
+Wire Wire Line
+	4550 3400 4900 3400
+Text Label 4650 3300 0    50   ~ 0
+RX-
+Text Label 4650 3400 0    50   ~ 0
+RX+
+$Comp
+L Device:C C45
+U 1 1 5C23D8BE
+P 8650 1900
+F 0 "C45" H 8450 1950 50  0000 L CNN
+F 1 "10nF" H 8350 1850 50  0000 L CNN
+F 2 "Capacitor_SMD:C_0603_1608Metric_Pad1.05x0.95mm_HandSolder" H 8688 1750 50  0001 C CNN
+F 3 "~" H 8650 1900 50  0001 C CNN
+	1    8650 1900
+	1    0    0    -1
+$EndComp
+Wire Wire Line
+	8650 2050 8650 2100
+Wire Wire Line
+	8650 2100 8300 2100
+Text Label 8350 2100 0    50   ~ 0
+AGND
+Wire Wire Line
+	9000 1600 8650 1600
+Wire Wire Line
+	8650 1600 8650 1750
+Connection ~ 9000 1600
+Wire Wire Line
+	1700 3700 1700 5450
+Connection ~ 1700 5450
+Wire Wire Line
+	1700 5450 1700 5500
+Wire Wire Line
+	900  3300 1200 3300
+$Comp
+L Device:R R65
+U 1 1 5C285117
+P 1200 3100
+F 0 "R65" H 1270 3146 50  0000 L CNN
+F 1 "10K" H 1270 3055 50  0000 L CNN
+F 2 "Resistor_SMD:R_0603_1608Metric_Pad1.05x0.95mm_HandSolder" V 1130 3100 50  0001 C CNN
+F 3 "~" H 1200 3100 50  0001 C CNN
+	1    1200 3100
+	1    0    0    -1
+$EndComp
+Wire Wire Line
+	1200 2900 1200 2950
+Wire Wire Line
+	1200 3250 1200 3300
+Connection ~ 1200 3300
+Wire Wire Line
+	1200 3300 2250 3300
 $EndSCHEMATC

Commit message: added footprints for Y3 FB1 FB3 FB2 F1
Parts:
- FB2, FB3: footprint (none) -> Inductor_SMD:L_0805_2012Metric_Pad1.15x1.40mm_HandSolder
- Y3: footprint (none) -> Crystal:Crystal_SMD_SeikoEpson_TSX3225-4Pin_3.2x2.5mm_HandSoldering
Changed lines of the file:
@@
 F 0 "Y3" H 1100 4418 50  0000 C CNN
 F 1 "25MHz" H 1100 4327 50  0000 C CNN
-F 2 "" H 1100 4150 50  0001 C CNN
+F 2 "Crystal:Crystal_SMD_SeikoEpson_TSX3225-4Pin_3.2x2.5mm_HandSoldering" H 1100 4150 50  0001 C CNN
 F 3 "~" H 1100 4150 50  0001 C CNN
 F 4 "EPSON" H 1100 4150 50  0001 C CNN "Manufacturer"
@@
 F 0 "FB2" V 4676 5900 50  0000 C CNN
 F 1 "Ferrite_Bead" V 4767 5900 50  0000 C CNN
-F 2 "" V 4880 5900 50  0001 C CNN
+F 2 "Inductor_SMD:L_0805_2012Metric_Pad1.15x1.40mm_HandSolder" V 4880 5900 50  0001 C CNN
 F 3 "~" H 4950 5900 50  0001 C CNN
 F 4 "Murata" V 4950 5900 50  0001 C CNN "Manufacturer"
@@
 F 0 "FB3" V 4676 6400 50  0000 C CNN
 F 1 "Ferrite_Bead" V 4767 6400 50  0000 C CNN
-F 2 "" V 4880 6400 50  0001 C CNN
+F 2 "Inductor_SMD:L_0805_2012Metric_Pad1.15x1.40mm_HandSolder" V 4880 6400 50  0001 C CNN
 F 3 "~" H 4950 6400 50  0001 C CNN
 F 4 "Murata" V 4950 6400 50  0001 C CNN "Manufacturer"

Commit message: updated motor drive circuitry, annotated
Other:
- note added: "Bypass resistor for MISO"
Changed lines of the file:
@@
 U 1 1 5C0721C1
 P 3400 3450
+AR Path="/5C0721C1" Ref="U8"  Part="1"
+AR Path="/5C06FA8E/5C0721C1" Ref="U8"  Part="1"
 F 0 "U8" H 4250 2450 50  0000 L CNN
 F 1 "W5500" H 2450 2450 50  0000 L CNN
@@
 Wire Wire Line
 	1200 3300 2250 3300
+Text Notes 2600 6400 0    50   ~ 0
+Bypass resistor for MISO
 $EndSCHEMATC

Commit message: added one resistor, about to rip up all traces and move all the parts around
Parts:
- added R87: OPEN, Resistor_SMD:R_0603_1608Metric_Pad1.05x0.95mm_HandSolder, symbol Device:R
Connections:
- wire segments 149 -> 154
Other:
- note added: "(Bypass resistor for MISO)"
- note removed: "Bypass resistor for MISO"
Changed lines of the file:
@@
 MISO_TRISTATE
 Wire Wire Line
-	600  7000 1300 7000
+	600  7000 700  7000
 Text HLabel 1200 6900 0    50   Input ~ 0
 CS
@@
 Wire Wire Line
 	1200 3300 2250 3300
-Text Notes 2600 6400 0    50   ~ 0
-Bypass resistor for MISO
+Text Notes 1100 7650 0    50   ~ 0
+(Bypass resistor for MISO)
+$Comp
+L Device:R R87
+U 1 1 5C32D791
+P 1550 7500
+F 0 "R87" V 1450 7450 50  0000 C CNN
+F 1 "OPEN" V 1550 7500 50  0000 C CNN
+F 2 "Resistor_SMD:R_0603_1608Metric_Pad1.05x0.95mm_HandSolder" V 1480 7500 50  0001 C CNN
+F 3 "~" H 1550 7500 50  0001 C CNN
+	1    1550 7500
+	0    1    1    0
+$EndComp
+Wire Wire Line
+	700  7000 700  7500
+Wire Wire Line
+	700  7500 1400 7500
+Connection ~ 700  7000
+Wire Wire Line
+	700  7000 1300 7000
+Wire Wire Line
+	1700 7500 2300 7500
+Wire Wire Line
+	2300 7500 2300 7100
+Connection ~ 2300 7100
 $EndSCHEMATC

Commit message: moving stuff around
Parts:
- Y3: symbol Device:Crystal -> Device:Crystal_GND24
Connections:
- wire segments 154 -> 157
Changed lines of the file:
@@
 	2250 3200 2100 3200
 $Comp
-L Device:Crystal Y3
+L Device:Crystal_GND24 Y3
 U 1 1 5C07687B
 P 1100 4150
-F 0 "Y3" H 1100 4418 50  0000 C CNN
-F 1 "25MHz" H 1100 4327 50  0000 C CNN
+F 0 "Y3" H 850 4300 50  0000 C CNN
+F 1 "25MHz" H 800 4200 50  0000 C CNN
 F 2 "Crystal:Crystal_SMD_SeikoEpson_TSX3225-4Pin_3.2x2.5mm_HandSoldering" H 1100 4150 50  0001 C CNN
 F 3 "~" H 1100 4150 50  0001 C CNN
@@
 U 1 1 5C07792B
 P 900 4500
-F 0 "C31" H 1015 4546 50  0000 L CNN
-F 1 "22pF" H 1015 4455 50  0000 L CNN
+F 0 "C31" H 650 4550 50  0000 L CNN
+F 1 "22pF" H 600 4450 50  0000 L CNN
 F 2 "Capacitor_SMD:C_0603_1608Metric_Pad1.05x0.95mm_HandSolder" H 938 4350 50  0001 C CNN
 F 3 "~" H 900 4500 50  0001 C CNN
@@
 Wire Wire Line
 	8600 3500 8600 3300
-Text Label 8600 4050 1    50   ~ 0
-AGND
-Wire Wire Line
-	8600 4050 8600 3800
+Text Label 8500 3850 2    50   ~ 0
+AGND
 $Comp
 L power:GND #PWR0129
@@
 U 1 1 5C23D8BE
 P 8650 1900
-F 0 "C45" H 8450 1950 50  0000 L CNN
+F 0 "C45" H 8400 1950 50  0000 L CNN
 F 1 "10nF" H 8350 1850 50  0000 L CNN
 F 2 "Capacitor_SMD:C_0603_1608Metric_Pad1.05x0.95mm_HandSolder" H 8688 1750 50  0001 C CNN
@@
 	2300 7500 2300 7100
 Connection ~ 2300 7100
+Wire Wire Line
+	8600 3850 8250 3850
+Wire Wire Line
+	8600 3850 8600 3800
+$Comp
+L power:GND #PWR?
+U 1 1 5C4380F9
+P 1100 4750
+F 0 "#PWR?" H 1100 4500 50  0001 C CNN
+F 1 "GND" H 1105 4577 50  0000 C CNN
+F 2 "" H 1100 4750 50  0001 C CNN
+F 3 "" H 1100 4750 50  0001 C CNN
+	1    1100 4750
+	1    0    0    -1
+$EndComp
+Wire Wire Line
+	1100 4350 1100 4750
+$Comp
+L power:GND #PWR?
+U 1 1 5C451215
+P 1100 3900
+F 0 "#PWR?" H 1100 3650 50  0001 C CNN
+F 1 "GND" H 1100 3750 50  0000 C CNN
+F 2 "" H 1100 3900 50  0001 C CNN
+F 3 "" H 1100 3900 50  0001 C CNN
+	1    1100 3900
+	-1   0    0    1
+$EndComp
+Wire Wire Line
+	1100 3900 1100 3950
 $EndSCHEMATC
