File: KiCad/motor_power.sch (KiCad schematic (older format))
At the start: 66 parts, among them Q10 N-CH 50V 200mA, Q11 N-CH 50V 200mA, Q12 P-CH 30V 3.8A, Q13 P-CH 30V 3.8A, Q14 Q_NMOS_SGD, Q15 Q_NMOS_SGD, Q16 N-CH 50V 200mA, Q17 N-CH 50V 200mA, Q18 P-CH 30V 3.8A, Q19 P-CH 30V 3.8A, Q2 Q_NMOS_SGD, Q20 Q_NMOS_SGD, Q21 Q_NMOS_SGD, Q22 N-CH 50V 200mA, Q23 N-CH 50V 200mA, Q24 P-CH 30V 3.8A, Q25 P-CH 30V 3.8A, Q3 Q_NMOS_SGD, Q4 N-CH 50V 200mA, Q5 N-CH 50V 200mA, Q6 P-CH 30V 3.8A, Q7 P-CH 30V 3.8A, Q8 Q_NMOS_SGD, Q9 Q_NMOS_SGD, U4 INA180B3, U5 INA219

Commit message: updated motor drive circuitry, annotated
Parts:
- removed Q10, Q11, Q16, Q17, Q22, Q23, Q4, Q5: N-CH 50V 200mA, Package_TO_SOT_SMD:TSOT-23_HandSoldering, symbol Device:Q_NMOS_GSD
- removed Q12, Q13, Q18, Q19, Q24, Q25, Q7: P-CH 30V 3.8A, Package_TO_SOT_SMD:TSOT-23_HandSoldering, symbol Device:Q_PMOS_GSD
- removed Q14, Q15, Q20, Q21, Q3, Q8, Q9: Q_NMOS_SGD, Package_TO_SOT_SMD:TSOT-23_HandSoldering, symbol Device:Q_NMOS_GSD
- removed R20, R29, R30, R39, R40, R47, R48: R, Resistor_SMD:R_0603_1608Metric_Pad1.05x0.95mm_HandSolder, symbol Device:R
- removed R22, R24, R25, R27, R31, R32, R34, R35, R36, R37, R41, R42, R43, R44, R45, R46, R49, R50, R51, R52, R53, R54: 1K, Resistor_SMD:R_0603_1608Metric_Pad1.05x0.95mm_HandSolder, symbol Device:R
- added C? (x8): 1uF 50V, symbol Device:C
- added D? (x8): 50V 2A, symbol Device:D
- added Q? (x8): MMBT3904, Package_TO_SOT_SMD:SOT-23_Handsoldering, symbol Transistor_BJT:MMBT3904
- added Q? (x7): P-CH 30V 3.8A, Package_TO_SOT_SMD:TSOT-23_HandSoldering, symbol Device:Q_PMOS_GSD
- added Q? (x7): Q_NMOS_SGD, Package_TO_SOT_SMD:TSOT-23_HandSoldering, symbol Device:Q_NMOS_GSD
- added R? (x15): 1K, Resistor_SMD:R_0603_1608Metric_Pad1.05x0.95mm_HandSolder, symbol Device:R
- added R? (x15): 1k, Resistor_SMD:R_0603_1608Metric_Pad1.05x0.95mm_HandSolder, symbol Device:R
- added R? (x7): 10k, Resistor_SMD:R_0603_1608Metric_Pad1.05x0.95mm_HandSolder, symbol Device:R
- R19: value R -> 1k
- R21: value 1K -> 10k
Connections:
- wire segments 209 -> 249
Other:
- moved on the sheet: C21, C22, JP1, JP2, Q6, R19, R21, R23, R26, R28, R33, R38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

Commit message: fixed S2A and motor drive capacitor footprint links
Parts:
- C46, C47, C48, C49, C50, C51, C52, C53: renamed from C?; footprint (none) -> Capacitor_SMD:C_0603_1608Metric_Pad1.05x0.95mm_HandSolder; Manufacturer (none) -> Samsung; Part Number (none) -> CL10A105KB8NNNC
- D1, D10, D11, D12, D13, D14, D3, D9: renamed from D?; footprint (none) -> Diode_SMD:D_SMB_Handsoldering
- gave numbers to parts that had none: 59

Commit message: Updated Schematic
Parts:
- D1, D10, D11, D12, D13, D14, D3, D9: footprint Diode_SMD:D_SMB_Handsoldering -> Snack Machine:D_SMB_Handsoldering_Lite
- Q10, Q15, Q16, Q17, Q18, Q7, Q8, Q9: footprint Package_TO_SOT_SMD:SOT-23_Handsoldering -> Snack Machine:SOT-23_Handsoldering_Lite
Changed lines of the file:
@@
 F 0 "Q7" H 2391 2246 50  0000 L CNN
 F 1 "MMBT3904" H 2391 2155 50  0000 L CNN
-F 2 "Package_TO_SOT_SMD:SOT-23_Handsoldering" H 2400 2125 50  0001 L CIN
+F 2 "Snack Machine:SOT-23_Handsoldering_Lite" H 2400 2125 50  0001 L CIN
 F 3 "https://www.fairchildsemi.com/datasheets/2N/2N3904.pdf" H 2200 2200 50  0001 L CNN
 	1    2200 2200
@@
 F 0 "Q8" H 5191 2246 50  0000 L CNN
 F 1 "MMBT3904" H 5191 2155 50  0000 L CNN
-F 2 "Package_TO_SOT_SMD:SOT-23_Handsoldering" H 5200 2125 50  0001 L CIN
+F 2 "Snack Machine:SOT-23_Handsoldering_Lite" H 5200 2125 50  0001 L CIN
 F 3 "https://www.fairchildsemi.com/datasheets/2N/2N3904.pdf" H 5000 2200 50  0001 L CNN
 	1    5000 2200
@@
 F 0 "D1" V 3050 1600 50  0000 L CNN
 F 1 "50V 2A" V 3150 1600 50  0000 L CNN
-F 2 "Diode_SMD:D_SMB_Handsoldering" H 3100 1500 50  0001 C CNN
+F 2 "Snack Machine:D_SMB_Handsoldering_Lite" H 3100 1500 50  0001 C CNN
 F 3 "~" H 3100 1500 50  0001 C CNN
 F 4 "ON Semiconductor" H 3100 1500 50  0001 C CNN "Manufacturer"
@@
 F 0 "D3" V 5850 1600 50  0000 L CNN
 F 1 "50V 2A" V 5950 1600 50  0000 L CNN
-F 2 "Diode_SMD:D_SMB_Handsoldering" H 5900 1500 50  0001 C CNN
+F 2 "Snack Machine:D_SMB_Handsoldering_Lite" H 5900 1500 50  0001 C CNN
 F 3 "~" H 5900 1500 50  0001 C CNN
 F 4 "ON Semiconductor" H 5900 1500 50  0001 C CNN "Manufacturer"
@@
 F 0 "Q9" H 7991 2246 50  0000 L CNN
 F 1 "MMBT3904" H 7991 2155 50  0000 L CNN
-F 2 "Package_TO_SOT_SMD:SOT-23_Handsoldering" H 8000 2125 50  0001 L CIN
+F 2 "Snack Machine:SOT-23_Handsoldering_Lite" H 8000 2125 50  0001 L CIN
 F 3 "https://www.fairchildsemi.com/datasheets/2N/2N3904.pdf" H 7800 2200 50  0001 L CNN
 	1    7800 2200
@@
 F 0 "Q10" H 10791 2246 50  0000 L CNN
 F 1 "MMBT3904" H 10791 2155 50  0000 L CNN
-F 2 "Package_TO_SOT_SMD:SOT-23_Handsoldering" H 10800 2125 50  0001 L CIN
+F 2 "Snack Machine:SOT-23_Handsoldering_Lite" H 10800 2125 50  0001 L CIN
 F 3 "https://www.fairchildsemi.com/datasheets/2N/2N3904.pdf" H 10600 2200 50  0001 L CNN
 	1    10600 2200
@@
 F 0 "D9" V 8650 1600 50  0000 L CNN
 F 1 "50V 2A" V 8750 1600 50  0000 L CNN
-F 2 "Diode_SMD:D_SMB_Handsoldering" H 8700 1500 50  0001 C CNN
+F 2 "Snack Machine:D_SMB_Handsoldering_Lite" H 8700 1500 50  0001 C CNN
 F 3 "~" H 8700 1500 50  0001 C CNN
 F 4 "ON Semiconductor" H 8700 1500 50  0001 C CNN "Manufacturer"
@@
 F 0 "D10" V 11450 1600 50  0000 L CNN
 F 1 "50V 2A" V 11550 1600 50  0000 L CNN
-F 2 "Diode_SMD:D_SMB_Handsoldering" H 11500 1500 50  0001 C CNN
+F 2 "Snack Machine:D_SMB_Handsoldering_Lite" H 11500 1500 50  0001 C CNN
 F 3 "~" H 11500 1500 50  0001 C CNN
 F 4 "ON Semiconductor" H 11500 1500 50  0001 C CNN "Manufacturer"
@@
 F 0 "Q15" H 2391 4196 50  0000 L CNN
 F 1 "MMBT3904" H 2391 4105 50  0000 L CNN
-F 2 "Package_TO_SOT_SMD:SOT-23_Handsoldering" H 2400 4075 50  0001 L CIN
+F 2 "Snack Machine:SOT-23_Handsoldering_Lite" H 2400 4075 50  0001 L CIN
 F 3 "https://www.fairchildsemi.com/datasheets/2N/2N3904.pdf" H 2200 4150 50  0001 L CNN
 	1    2200 4150
@@
 F 0 "Q16" H 5191 4196 50  0000 L CNN
 F 1 "MMBT3904" H 5191 4105 50  0000 L CNN
-F 2 "Package_TO_SOT_SMD:SOT-23_Handsoldering" H 5200 4075 50  0001 L CIN
+F 2 "Snack Machine:SOT-23_Handsoldering_Lite" H 5200 4075 50  0001 L CIN
 F 3 "https://www.fairchildsemi.com/datasheets/2N/2N3904.pdf" H 5000 4150 50  0001 L CNN
 	1    5000 4150
@@
 F 0 "D11" V 3050 3550 50  0000 L CNN
 F 1 "50V 2A" V 3150 3550 50  0000 L CNN
-F 2 "Diode_SMD:D_SMB_Handsoldering" H 3100 3450 50  0001 C CNN
+F 2 "Snack Machine:D_SMB_Handsoldering_Lite" H 3100 3450 50  0001 C CNN
 F 3 "~" H 3100 3450 50  0001 C CNN
 F 4 "ON Semiconductor" H 3100 3450 50  0001 C CNN "Manufacturer"
@@
 F 0 "D12" V 5850 3550 50  0000 L CNN
 F 1 "50V 2A" V 5950 3550 50  0000 L CNN
-F 2 "Diode_SMD:D_SMB_Handsoldering" H 5900 3450 50  0001 C CNN
+F 2 "Snack Machine:D_SMB_Handsoldering_Lite" H 5900 3450 50  0001 C CNN
 F 3 "~" H 5900 3450 50  0001 C CNN
 F 4 "ON Semiconductor" H 5900 3450 50  0001 C CNN "Manufacturer"
@@
 F 0 "Q17" H 7991 4196 50  0000 L CNN
 F 1 "MMBT3904" H 7991 4105 50  0000 L CNN
-F 2 "Package_TO_SOT_SMD:SOT-23_Handsoldering" H 8000 4075 50  0001 L CIN
+F 2 "Snack Machine:SOT-23_Handsoldering_Lite" H 8000 4075 50  0001 L CIN
 F 3 "https://www.fairchildsemi.com/datasheets/2N/2N3904.pdf" H 7800 4150 50  0001 L CNN
 	1    7800 4150
@@
 F 0 "Q18" H 10791 4196 50  0000 L CNN
 F 1 "MMBT3904" H 10791 4105 50  0000 L CNN
-F 2 "Package_TO_SOT_SMD:SOT-23_Handsoldering" H 10800 4075 50  0001 L CIN
+F 2 "Snack Machine:SOT-23_Handsoldering_Lite" H 10800 4075 50  0001 L CIN
 F 3 "https://www.fairchildsemi.com/datasheets/2N/2N3904.pdf" H 10600 4150 50  0001 L CNN
 	1    10600 4150
@@
 F 0 "D13" V 8650 3550 50  0000 L CNN
 F 1 "50V 2A" V 8750 3550 50  0000 L CNN
-F 2 "Diode_SMD:D_SMB_Handsoldering" H 8700 3450 50  0001 C CNN
+F 2 "Snack Machine:D_SMB_Handsoldering_Lite" H 8700 3450 50  0001 C CNN
 F 3 "~" H 8700 3450 50  0001 C CNN
 F 4 "ON Semiconductor" H 8700 3450 50  0001 C CNN "Manufacturer"
@@
 F 0 "D14" V 11450 3550 50  0000 L CNN
 F 1 "50V 2A" V 11550 3550 50  0000 L CNN
-F 2 "Diode_SMD:D_SMB_Handsoldering" H 11500 3450 50  0001 C CNN
+F 2 "Snack Machine:D_SMB_Handsoldering_Lite" H 11500 3450 50  0001 C CNN
 F 3 "~" H 11500 3450 50  0001 C CNN
 F 4 "ON Semiconductor" H 11500 3450 50  0001 C CNN "Manufacturer"

Commit message: changed footprint for TSOT23 handsoldering to be more reasonable
Parts:
- Q11, Q12, Q13, Q14, Q19, Q2, Q20, Q21, Q22, Q23, Q24, Q25, Q3, Q4, Q5, Q6: footprint Package_TO_SOT_SMD:TSOT-23_HandSoldering -> Snack Machine:TSOT-23_HandSoldering_Lite
Changed lines of the file:
@@
 F 0 "Q6" V 2650 1300 50  0000 L CNN
 F 1 "P-CH 30V 3.8A" V 2550 1300 50  0000 L CNN
-F 2 "Package_TO_SOT_SMD:TSOT-23_HandSoldering" H 2500 1450 50  0001 C CNN
+F 2 "Snack Machine:TSOT-23_HandSoldering_Lite" H 2500 1450 50  0001 C CNN
 F 3 "~" H 2300 1350 50  0001 C CNN
 F 4 "Diodes Incorporated" V 2300 1350 50  0001 C CNN "Manufacturer"
@@
 F 0 "Q2" H 2405 5246 50  0000 L CNN
 F 1 "Q_NMOS_SGD" H 2405 5155 50  0000 L CNN
-F 2 "Package_TO_SOT_SMD:TSOT-23_HandSoldering" H 2400 5300 50  0001 C CNN
+F 2 "Snack Machine:TSOT-23_HandSoldering_Lite" H 2400 5300 50  0001 C CNN
 F 3 "~" H 2200 5200 50  0001 C CNN
 F 4 "ON Semiconductor" H 2200 5200 50  0001 C CNN "Manufacturer"
@@
 F 0 "Q3" V 5450 1300 50  0000 L CNN
 F 1 "P-CH 30V 3.8A" V 5350 1300 50  0000 L CNN
-F 2 "Package_TO_SOT_SMD:TSOT-23_HandSoldering" H 5300 1450 50  0001 C CNN
+F 2 "Snack Machine:TSOT-23_HandSoldering_Lite" H 5300 1450 50  0001 C CNN
 F 3 "~" H 5100 1350 50  0001 C CNN
 F 4 "Diodes Incorporated" V 5100 1350 50  0001 C CNN "Manufacturer"
@@
 F 0 "Q4" V 8250 1300 50  0000 L CNN
 F 1 "P-CH 30V 3.8A" V 8150 1300 50  0000 L CNN
-F 2 "Package_TO_SOT_SMD:TSOT-23_HandSoldering" H 8100 1450 50  0001 C CNN
+F 2 "Snack Machine:TSOT-23_HandSoldering_Lite" H 8100 1450 50  0001 C CNN
 F 3 "~" H 7900 1350 50  0001 C CNN
 F 4 "Diodes Incorporated" V 7900 1350 50  0001 C CNN "Manufacturer"
@@
 F 0 "Q5" V 11050 1300 50  0000 L CNN
 F 1 "P-CH 30V 3.8A" V 10950 1300 50  0000 L CNN
-F 2 "Package_TO_SOT_SMD:TSOT-23_HandSoldering" H 10900 1450 50  0001 C CNN
+F 2 "Snack Machine:TSOT-23_HandSoldering_Lite" H 10900 1450 50  0001 C CNN
 F 3 "~" H 10700 1350 50  0001 C CNN
 F 4 "Diodes Incorporated" V 10700 1350 50  0001 C CNN "Manufacturer"
@@
 F 0 "Q11" V 2650 3250 50  0000 L CNN
 F 1 "P-CH 30V 3.8A" V 2550 3250 50  0000 L CNN
-F 2 "Package_TO_SOT_SMD:TSOT-23_HandSoldering" H 2500 3400 50  0001 C CNN
+F 2 "Snack Machine:TSOT-23_HandSoldering_Lite" H 2500 3400 50  0001 C CNN
 F 3 "~" H 2300 3300 50  0001 C CNN
 F 4 "Diodes Incorporated" V 2300 3300 50  0001 C CNN "Manufacturer"
@@
 F 0 "Q12" V 5450 3250 50  0000 L CNN
 F 1 "P-CH 30V 3.8A" V 5350 3250 50  0000 L CNN
-F 2 "Package_TO_SOT_SMD:TSOT-23_HandSoldering" H 5300 3400 50  0001 C CNN
+F 2 "Snack Machine:TSOT-23_HandSoldering_Lite" H 5300 3400 50  0001 C CNN
 F 3 "~" H 5100 3300 50  0001 C CNN
 F 4 "Diodes Incorporated" V 5100 3300 50  0001 C CNN "Manufacturer"
@@
 F 0 "Q13" V 8250 3250 50  0000 L CNN
 F 1 "P-CH 30V 3.8A" V 8150 3250 50  0000 L CNN
-F 2 "Package_TO_SOT_SMD:TSOT-23_HandSoldering" H 8100 3400 50  0001 C CNN
+F 2 "Snack Machine:TSOT-23_HandSoldering_Lite" H 8100 3400 50  0001 C CNN
 F 3 "~" H 7900 3300 50  0001 C CNN
 F 4 "Diodes Incorporated" V 7900 3300 50  0001 C CNN "Manufacturer"
@@
 F 0 "Q14" V 11050 3250 50  0000 L CNN
 F 1 "P-CH 30V 3.8A" V 10950 3250 50  0000 L CNN
-F 2 "Package_TO_SOT_SMD:TSOT-23_HandSoldering" H 10900 3400 50  0001 C CNN
+F 2 "Snack Machine:TSOT-23_HandSoldering_Lite" H 10900 3400 50  0001 C CNN
 F 3 "~" H 10700 3300 50  0001 C CNN
 F 4 "Diodes Incorporated" V 10700 3300 50  0001 C CNN "Manufacturer"
@@
 F 0 "Q19" H 5205 5246 50  0000 L CNN
 F 1 "Q_NMOS_SGD" H 5205 5155 50  0000 L CNN
-F 2 "Package_TO_SOT_SMD:TSOT-23_HandSoldering" H 5200 5300 50  0001 C CNN
+F 2 "Snack Machine:TSOT-23_HandSoldering_Lite" H 5200 5300 50  0001 C CNN
 F 3 "~" H 5000 5200 50  0001 C CNN
 F 4 "ON Semiconductor" H 5000 5200 50  0001 C CNN "Manufacturer"
@@
 F 0 "Q20" H 8005 5246 50  0000 L CNN
 F 1 "Q_NMOS_SGD" H 8005 5155 50  0000 L CNN
-F 2 "Package_TO_SOT_SMD:TSOT-23_HandSoldering" H 8000 5300 50  0001 C CNN
+F 2 "Snack Machine:TSOT-23_HandSoldering_Lite" H 8000 5300 50  0001 C CNN
 F 3 "~" H 7800 5200 50  0001 C CNN
 F 4 "ON Semiconductor" H 7800 5200 50  0001 C CNN "Manufacturer"
@@
 F 0 "Q21" H 10805 5246 50  0000 L CNN
 F 1 "Q_NMOS_SGD" H 10805 5155 50  0000 L CNN
-F 2 "Package_TO_SOT_SMD:TSOT-23_HandSoldering" H 10800 5300 50  0001 C CNN
+F 2 "Snack Machine:TSOT-23_HandSoldering_Lite" H 10800 5300 50  0001 C CNN
 F 3 "~" H 10600 5200 50  0001 C CNN
 F 4 "ON Semiconductor" H 10600 5200 50  0001 C CNN "Manufacturer"
@@
 F 0 "Q22" H 2405 6346 50  0000 L CNN
 F 1 "Q_NMOS_SGD" H 2405 6255 50  0000 L CNN
-F 2 "Package_TO_SOT_SMD:TSOT-23_HandSoldering" H 2400 6400 50  0001 C CNN
+F 2 "Snack Machine:TSOT-23_HandSoldering_Lite" H 2400 6400 50  0001 C CNN
 F 3 "~" H 2200 6300 50  0001 C CNN
 F 4 "ON Semiconductor" H 2200 6300 50  0001 C CNN "Manufacturer"
@@
 F 0 "Q23" H 5205 6346 50  0000 L CNN
 F 1 "Q_NMOS_SGD" H 5205 6255 50  0000 L CNN
-F 2 "Package_TO_SOT_SMD:TSOT-23_HandSoldering" H 5200 6400 50  0001 C CNN
+F 2 "Snack Machine:TSOT-23_HandSoldering_Lite" H 5200 6400 50  0001 C CNN
 F 3 "~" H 5000 6300 50  0001 C CNN
 F 4 "ON Semiconductor" H 5000 6300 50  0001 C CNN "Manufacturer"
@@
 F 0 "Q24" H 8005 6346 50  0000 L CNN
 F 1 "Q_NMOS_SGD" H 8005 6255 50  0000 L CNN
-F 2 "Package_TO_SOT_SMD:TSOT-23_HandSoldering" H 8000 6400 50  0001 C CNN
+F 2 "Snack Machine:TSOT-23_HandSoldering_Lite" H 8000 6400 50  0001 C CNN
 F 3 "~" H 7800 6300 50  0001 C CNN
 F 4 "ON Semiconductor" H 7800 6300 50  0001 C CNN "Manufacturer"
@@
 F 0 "Q25" H 10805 6346 50  0000 L CNN
 F 1 "Q_NMOS_SGD" H 10805 6255 50  0000 L CNN
-F 2 "Package_TO_SOT_SMD:TSOT-23_HandSoldering" H 10800 6400 50  0001 C CNN
+F 2 "Snack Machine:TSOT-23_HandSoldering_Lite" H 10800 6400 50  0001 C CNN
 F 3 "~" H 10600 6300 50  0001 C CNN
 F 4 "ON Semiconductor" H 10600 6300 50  0001 C CNN "Manufacturer"

Commit message: Updating a ton of part numbers
Parts:
- C21, C22: value 0.1uF -> 100nF; Manufacturer (none) -> Yageo; Part Number (none) -> CC0603KRX7R9BB104
- Q10: Manufacturer (none) -> MCC; Part Numberr (none) -> MMBT3904-TP
- Q15, Q16, Q17, Q18, Q7, Q8, Q9: Manufacturer (none) -> MCC; Part Number (none) -> MMBT3904-TP
- R19, R31, R32, R34, R44, R45, R46, R47, R48, R49, R50, R51, R79, R80, R81, R82: Manufacturer (none) -> Yageo; Part Number (none) -> RC0603FR-071KL
- R20, R22, R24, R25, R26, R27, R29, R30, R35, R36, R37, R39, R40, R41, R42, R43: value 1K -> 1k; Manufacturer (none) -> Yageo; Part Number (none) -> RC0603FR-071KL
- R21, R28, R33, R52, R53, R54, R83, R84, R85, R86: Manufacturer (none) -> Yageo; Part Number (none) -> RC0603FR-0710KL
- R23, R38: Manufacturer (none) -> Samsung; Part Number (none) -> RUT2012FR100CS
- U5: Manufacturer (none) -> Texas Instruments; Part Number (none) -> INA219AIDCNR

Commit message: Fixing small typo
Parts:
- Q10: Part Number (none) -> MMBT3904-TP; Part Numberr MMBT3904-TP -> (none)
Changed lines of the file:
@@
 F 2 "Snack Machine:SOT-23_Handsoldering_Lite" H 10800 2125 50  0001 L CIN
 F 3 "https://www.fairchildsemi.com/datasheets/2N/2N3904.pdf" H 10600 2200 50  0001 L CNN
-F 4 "MMBT3904-TP" H 10600 2200 50  0001 C CNN "Part Numberr"
+F 4 "MMBT3904-TP" H 10600 2200 50  0001 C CNN "Part Number"
 F 5 "MCC" H 10600 2200 50  0001 C CNN "Manufacturer"
 	1    10600 2200

Commit message: Making a bunch of changes throughout the board
Parts:
- removed C21, C22: 100nF, Capacitor_SMD:C_0603_1608Metric_Pad1.05x0.95mm_HandSolder, symbol Device:C
- removed C46, C47, C48, C49, C50, C51, C52, C53: 1uF 50V, Capacitor_SMD:C_0603_1608Metric_Pad1.05x0.95mm_HandSolder, symbol Device:C
- removed D1, D10, D11, D12, D13, D14, D3, D9: 50V 2A, Snack Machine:D_SMB_Handsoldering_Lite, symbol Device:D
- removed JP1, JP2: SolderJumper_2_Open, Jumper:SolderJumper-2_P1.3mm_Open_TrianglePad1.0x1.5mm, symbol Jumper:SolderJumper_2_Open
- removed Q10, Q15, Q16, Q17, Q18, Q7, Q8, Q9: MMBT3904, Snack Machine:SOT-23_Handsoldering_Lite, symbol Transistor_BJT:MMBT3904
- removed Q11, Q12, Q13, Q14, Q3, Q4, Q5, Q6: P-CH 30V 3.8A, Snack Machine:TSOT-23_HandSoldering_Lite, symbol Device:Q_PMOS_GSD
- removed Q19, Q2, Q20, Q21, Q22, Q23, Q24, Q25: Q_NMOS_SGD, Snack Machine:TSOT-23_HandSoldering_Lite, symbol Device:Q_NMOS_GSD
- removed R19, R20, R22, R24, R25, R26, R27, R29, R30, R31, R32, R34, R35, R36, R37, R39, R40, R41, R42, R43, R44, R45, R46, R47, R48, R49, R50, R51, R79, R80, R81, R82: 1k, Resistor_SMD:R_0603_1608Metric_Pad1.05x0.95mm_HandSolder, symbol Device:R
- removed R21, R28, R33, R52, R53, R54, R83, R84, R85, R86: 10k, Resistor_SMD:R_0603_1608Metric_Pad1.05x0.95mm_HandSolder, symbol Device:R
- removed R23, R38: 0.1R 1%, Resistor_SMD:R_0805_2012Metric_Pad1.15x1.40mm_HandSolder, symbol Device:R
- removed U4: INA180B3, Package_TO_SOT_SMD:SOT-23-5_HandSoldering, symbol Snack_Machine:INA180B3
- removed U5: INA219, Package_TO_SOT_SMD:TSOT-23-8_HandSoldering, symbol Snack_Machine:INA219
- added C? (x2): 2.2 uF, symbol Device:C
- added C?: 220 uF, symbol Device:CP
- added C? (x2): 100 nF, symbol Device:C
- added C?: 1 nF, symbol Device:C
- added D?: S1GTR, symbol Device:D
- added D? (x8): Q_TRIAC_A1A2G, symbol Device:Q_TRIAC_A1A2G
- added R?: 330 k, symbol Device:R
- added R?: 270 k, symbol Device:R
- added R?: 100 k, symbol Device:R
- added R? (x8): 1 k, symbol Device:R
- added U?: TBD62783A, symbol Transistor_Array:TBD62783A
- added U?: DPS1133FIA-13, kicad_pcb:QFN-17-Diodes1, symbol Snack_Machine:DPS1133FIA-13
Connections:
- net labels added: MOTOR_FAULT
- net labels removed: +5V, SCL, SDA, col_6_ctrl, motor_common_gnd
- wire segments 249 -> 43
Other:
- note added: "10 uA / A\n1 V/A with 100k"
- note removed: "High Side\nMotor Driving"
- note removed: "Low Side\nMotor Driving"
