File: KiCad/motor_power.sch (KiCad schematic (older format))
At the start: 29 parts, among them U1 DPS1133FIA-13, U4 TBD62783A

Commit message: Added part number, manufacturer, and personal bin numbers
Parts:
- C2: Bin (none) -> 32; Manufacturer (none) -> Taiyo Yuden
- C21, C6: Bin (none) -> 2; Manufacturer (none) -> Yageo; Part Number (none) -> CC0603KRX7R9BB104
- C22, C4: Bin (none) -> 25; Manufacturer (none) -> TDK
- C8: Bin (none) -> 35; Manufacturer (none) -> TDK
- D1, D10, D11, D12, D13, D14, D3, D9: Bin (none) -> 27; Manufacturer (none) -> WeEn Semiconductors; Part Number (none) -> Z0103MN,135
- D15: Bin (none) -> 29; Manufacturer (none) -> SMC Diode Solutions; Part Number (none) -> S1GTR
- R17, R19, R2, R20, R21, R22, R31, R8, R9: Bin (none) -> 1; Manufacturer (none) -> Yageo; Part Number (none) -> RC0603FR-071KL
- R18: Bin (none) -> 20; Manufacturer (none) -> Yageo; Part Number (none) -> RC0603FR-07330KL
- R23: Bin (none) -> 21; Manufacturer (none) -> Yageo; Part Number (none) -> RC0603FR-07270KL
- R24: Bin (none) -> 16; Manufacturer (none) -> Yageo; Part Number (none) -> RC0603FR-07100KL
- U1: Bin (none) -> 33; Manufacturer (none) -> Diodes Incorporated; Part Number (none) -> DPS1133FIA-13
- U4: Bin (none) -> 34; Manufacturer (none) -> Toshiba Semiconductor and Storage; Part Number (none) -> TBD62783AFNG,EL
Changed lines of the file:
@@
 F 2 "Package_SO:SSOP-18_4.4x6.5mm_P0.65mm" H 6450 900 50  0001 C CNN
 F 3 "http://toshiba.semicon-storage.com/info/docget.jsp?did=30523&prodName=TBD62783APG" H 6150 1850 50  0001 C CNN
+F 4 "TBD62783AFNG,EL" H 6450 1450 50  0001 C CNN "Part Number"
+F 5 "Toshiba Semiconductor and Storage" H 6450 1450 50  0001 C CNN "Manufacturer"
+F 6 "34" H 6450 1450 50  0001 C CNN "Bin"
 	1    6450 1450
 	1    0    0    -1
@@
 F 2 "Snack Machine:DPS1133FIA-13" H 2450 1200 50  0001 L CNN
 F 3 "" V 2700 1150 50  0001 C CNN
+F 4 "DPS1133FIA-13" H 2450 1150 50  0001 C CNN "Part Number"
+F 5 "Diodes Incorporated" H 2450 1150 50  0001 C CNN "Manufacturer"
+F 6 "33" H 2450 1150 50  0001 C CNN "Bin"
 	1    2450 1150
 	1    0    0    -1
@@
 F 3 "~" H 1550 1000 50  0001 C CNN
 F 4 "C1608JB1V225K080AC" H 1550 1000 50  0001 C CNN "Part Number"
+F 5 "TDK" H 1550 1000 50  0001 C CNN "Manufacturer"
+F 6 "25" H 1550 1000 50  0001 C CNN "Bin"
 	1    1550 1000
 	1    0    0    -1
@@
 F 2 "Capacitor_SMD:C_0603_1608Metric_Pad1.05x0.95mm_HandSolder" H 2038 2100 50  0001 C CNN
 F 3 "~" H 2000 2250 50  0001 C CNN
+F 4 "CC0603KRX7R9BB104" H 2000 2250 50  0001 C CNN "Part Number"
+F 5 "Yageo" H 2000 2250 50  0001 C CNN "Manufacturer"
+F 6 "2" H 2000 2250 50  0001 C CNN "Bin"
 	1    2000 2250
 	1    0    0    -1
@@
 F 3 "~" H 3250 2100 50  0001 C CNN
 F 4 "C1608C0G1H102J080AA" H 3250 2100 50  0001 C CNN "Part Number"
+F 5 "TDK" H 3250 2100 50  0001 C CNN "Manufacturer"
+F 6 "35" H 3250 2100 50  0001 C CNN "Bin"
 	1    3250 2100
 	1    0    0    -1
@@
 F 2 "Resistor_SMD:R_0603_1608Metric_Pad1.05x0.95mm_HandSolder" V 3630 1900 50  0001 C CNN
 F 3 "~" H 3700 1900 50  0001 C CNN
+F 4 "RC0603FR-07330KL" H 3700 1900 50  0001 C CNN "Part Number"
+F 5 "Yageo" H 3700 1900 50  0001 C CNN "Manufacturer"
+F 6 "20" H 3700 1900 50  0001 C CNN "Bin"
 	1    3700 1900
 	1    0    0    -1
@@
 F 2 "Resistor_SMD:R_0603_1608Metric_Pad1.05x0.95mm_HandSolder" V 4030 1800 50  0001 C CNN
 F 3 "~" H 4100 1800 50  0001 C CNN
+F 4 "RC0603FR-07270KL" H 4100 1800 50  0001 C CNN "Part Number"
+F 5 "Yageo" H 4100 1800 50  0001 C CNN "Manufacturer"
+F 6 "21" H 4100 1800 50  0001 C CNN "Bin"
 	1    4100 1800
 	1    0    0    -1
@@
 F 2 "Resistor_SMD:R_0603_1608Metric_Pad1.05x0.95mm_HandSolder" V 4430 2450 50  0001 C CNN
 F 3 "~" H 4500 2450 50  0001 C CNN
+F 4 "RC0603FR-07100KL" H 4500 2450 50  0001 C CNN "Part Number"
+F 5 "Yageo" H 4500 2450 50  0001 C CNN "Manufacturer"
+F 6 "16" H 4500 2450 50  0001 C CNN "Bin"
 	1    4500 2450
 	1    0    0    -1
@@
 F 2 "Capacitor_SMD:C_0603_1608Metric_Pad1.05x0.95mm_HandSolder" H 4088 2300 50  0001 C CNN
 F 3 "~" H 4050 2450 50  0001 C CNN
+F 4 "CC0603KRX7R9BB104" H 4050 2450 50  0001 C CNN "Part Number"
+F 5 "Yageo" H 4050 2450 50  0001 C CNN "Manufacturer"
+F 6 "2" H 4050 2450 50  0001 C CNN "Bin"
 	1    4050 2450
 	1    0    0    -1
@@
 F 2 "Diode_SMD:D_SMA_Handsoldering" H 4850 950 50  0001 C CNN
 F 3 "~" H 4850 950 50  0001 C CNN
+F 4 "S1GTR" H 4850 950 50  0001 C CNN "Part Number"
+F 5 "SMC Diode Solutions" H 4850 950 50  0001 C CNN "Manufacturer"
+F 6 "29" H 4850 950 50  0001 C CNN "Bin"
 	1    4850 950
 	1    0    0    -1
@@
 F 3 "~" H 5000 1400 50  0001 C CNN
 F 4 "C1608JB1V225K080AC" H 5000 1400 50  0001 C CNN "Part Number"
+F 5 "TDK" H 5000 1400 50  0001 C CNN "Manufacturer"
+F 6 "25" H 5000 1400 50  0001 C CNN "Bin"
 	1    5000 1400
 	1    0    0    -1
@@
 F 2 "Package_TO_SOT_SMD:SOT-223-3_TabPin2" V 1825 3125 50  0001 C CNN
 F 3 "~" V 1750 3100 50  0001 C CNN
+F 4 "Z0103MN,135" H 1750 3100 50  0001 C CNN "Part Number"
+F 5 "WeEn Semiconductors" H 1750 3100 50  0001 C CNN "Manufacturer"
+F 6 "27" H 1750 3100 50  0001 C CNN "Bin"
 	1    1750 3100
 	1    0    0    -1
@@
 F 2 "Resistor_SMD:R_0603_1608Metric_Pad1.05x0.95mm_HandSolder" V 1130 3200 50  0001 C CNN
 F 3 "~" H 1200 3200 50  0001 C CNN
+F 4 "RC0603FR-071KL" V 1200 3200 50  0001 C CNN "Part Number"
+F 5 "Yageo" V 1200 3200 50  0001 C CNN "Manufacturer"
+F 6 "1" V 1200 3200 50  0001 C CNN "Bin"
 	1    1200 3200
 	0    -1   -1   0
@@
 F 2 "Package_TO_SOT_SMD:SOT-223-3_TabPin2" V 1825 3775 50  0001 C CNN
 F 3 "~" V 1750 3750 50  0001 C CNN
+F 4 "Z0103MN,135" H 1750 3750 50  0001 C CNN "Part Number"
+F 5 "WeEn Semiconductors" H 1750 3750 50  0001 C CNN "Manufacturer"
+F 6 "27" H 1750 3750 50  0001 C CNN "Bin"
 	1    1750 3750
 	1    0    0    -1
@@
 F 2 "Resistor_SMD:R_0603_1608Metric_Pad1.05x0.95mm_HandSolder" V 1130 3850 50  0001 C CNN
 F 3 "~" H 1200 3850 50  0001 C CNN
+F 4 "RC0603FR-071KL" V 1200 3850 50  0001 C CNN "Part Number"
+F 5 "Yageo" V 1200 3850 50  0001 C CNN "Manufacturer"
+F 6 "1" V 1200 3850 50  0001 C CNN "Bin"
 	1    1200 3850
 	0    -1   -1   0
@@
 F 2 "Package_TO_SOT_SMD:SOT-223-3_TabPin2" V 1825 4425 50  0001 C CNN
 F 3 "~" V 1750 4400 50  0001 C CNN
+F 4 "Z0103MN,135" H 1750 4400 50  0001 C CNN "Part Number"
+F 5 "WeEn Semiconductors" H 1750 4400 50  0001 C CNN "Manufacturer"
+F 6 "27" H 1750 4400 50  0001 C CNN "Bin"
 	1    1750 4400
 	1    0    0    -1
@@
 F 2 "Resistor_SMD:R_0603_1608Metric_Pad1.05x0.95mm_HandSolder" V 1130 4500 50  0001 C CNN
 F 3 "~" H 1200 4500 50  0001 C CNN
+F 4 "RC0603FR-071KL" V 1200 4500 50  0001 C CNN "Part Number"
+F 5 "Yageo" V 1200 4500 50  0001 C CNN "Manufacturer"
+F 6 "1" V 1200 4500 50  0001 C CNN "Bin"
 	1    1200 4500
 	0    -1   -1   0
@@
 F 2 "Package_TO_SOT_SMD:SOT-223-3_TabPin2" V 1825 5075 50  0001 C CNN
 F 3 "~" V 1750 5050 50  0001 C CNN
+F 4 "Z0103MN,135" H 1750 5050 50  0001 C CNN "Part Number"
+F 5 "WeEn Semiconductors" H 1750 5050 50  0001 C CNN "Manufacturer"
+F 6 "27" H 1750 5050 50  0001 C CNN "Bin"
 	1    1750 5050
 	1    0    0    -1
@@
 F 2 "Resistor_SMD:R_0603_1608Metric_Pad1.05x0.95mm_HandSolder" V 1130 5150 50  0001 C CNN
 F 3 "~" H 1200 5150 50  0001 C CNN
+F 4 "RC0603FR-071KL" V 1200 5150 50  0001 C CNN "Part Number"
+F 5 "Yageo" V 1200 5150 50  0001 C CNN "Manufacturer"
+F 6 "1" V 1200 5150 50  0001 C CNN "Bin"
 	1    1200 5150
 	0    -1   -1   0
@@
 F 2 "Package_TO_SOT_SMD:SOT-223-3_TabPin2" V 4425 3125 50  0001 C CNN
 F 3 "~" V 4350 3100 50  0001 C CNN
+F 4 "Z0103MN,135" H 4350 3100 50  0001 C CNN "Part Number"
+F 5 "WeEn Semiconductors" H 4350 3100 50  0001 C CNN "Manufacturer"
+F 6 "27" H 4350 3100 50  0001 C CNN "Bin"
 	1    4350 3100
 	1    0    0    -1
@@
 F 2 "Resistor_SMD:R_0603_1608Metric_Pad1.05x0.95mm_HandSolder" V 3730 3200 50  0001 C CNN
 F 3 "~" H 3800 3200 50  0001 C CNN
+F 4 "RC0603FR-071KL" V 3800 3200 50  0001 C CNN "Part Number"
+F 5 "Yageo" V 3800 3200 50  0001 C CNN "Manufacturer"
+F 6 "1" V 3800 3200 50  0001 C CNN "Bin"
 	1    3800 3200
 	0    -1   -1   0
@@
 F 2 "Package_TO_SOT_SMD:SOT-223-3_TabPin2" V 4425 3775 50  0001 C CNN
 F 3 "~" V 4350 3750 50  0001 C CNN
+F 4 "Z0103MN,135" H 4350 3750 50  0001 C CNN "Part Number"
+F 5 "WeEn Semiconductors" H 4350 3750 50  0001 C CNN "Manufacturer"
+F 6 "27" H 4350 3750 50  0001 C CNN "Bin"
 	1    4350 3750
 	1    0    0    -1
@@
 F 2 "Resistor_SMD:R_0603_1608Metric_Pad1.05x0.95mm_HandSolder" V 3730 3850 50  0001 C CNN
 F 3 "~" H 3800 3850 50  0001 C CNN
+F 4 "RC0603FR-071KL" V 3800 3850 50  0001 C CNN "Part Number"
+F 5 "Yageo" V 3800 3850 50  0001 C CNN "Manufacturer"
+F 6 "1" V 3800 3850 50  0001 C CNN "Bin"
 	1    3800 3850
 	0    -1   -1   0
@@
 F 2 "Package_TO_SOT_SMD:SOT-223-3_TabPin2" V 4425 4425 50  0001 C CNN
 F 3 "~" V 4350 4400 50  0001 C CNN
+F 4 "Z0103MN,135" H 4350 4400 50  0001 C CNN "Part Number"
+F 5 "WeEn Semiconductors" H 4350 4400 50  0001 C CNN "Manufacturer"
+F 6 "27" H 4350 4400 50  0001 C CNN "Bin"
 	1    4350 4400
 	1    0    0    -1
@@
 F 2 "Resistor_SMD:R_0603_1608Metric_Pad1.05x0.95mm_HandSolder" V 3730 4500 50  0001 C CNN
 F 3 "~" H 3800 4500 50  0001 C CNN
+F 4 "RC0603FR-071KL" V 3800 4500 50  0001 C CNN "Part Number"
+F 5 "Yageo" V 3800 4500 50  0001 C CNN "Manufacturer"
+F 6 "1" V 3800 4500 50  0001 C CNN "Bin"
 	1    3800 4500
 	0    -1   -1   0
@@
 F 2 "Package_TO_SOT_SMD:SOT-223-3_TabPin2" V 4425 5075 50  0001 C CNN
 F 3 "~" V 4350 5050 50  0001 C CNN
+F 4 "Z0103MN,135" H 4350 5050 50  0001 C CNN "Part Number"
+F 5 "WeEn Semiconductors" H 4350 5050 50  0001 C CNN "Manufacturer"
+F 6 "27" H 4350 5050 50  0001 C CNN "Bin"
 	1    4350 5050
 	1    0    0    -1
@@
 F 2 "Resistor_SMD:R_0603_1608Metric_Pad1.05x0.95mm_HandSolder" V 3730 5150 50  0001 C CNN
 F 3 "~" H 3800 5150 50  0001 C CNN
+F 4 "RC0603FR-071KL" V 3800 5150 50  0001 C CNN "Part Number"
+F 5 "Yageo" V 3800 5150 50  0001 C CNN "Manufacturer"
+F 6 "1" V 3800 5150 50  0001 C CNN "Bin"
 	1    3800 5150
 	0    -1   -1   0
@@
 F 2 "Resistor_SMD:R_0603_1608Metric_Pad1.05x0.95mm_HandSolder" V 3330 850 50  0001 C CNN
 F 3 "~" H 3400 850 50  0001 C CNN
+F 4 "RC0603FR-071KL" H 3400 850 50  0001 C CNN "Part Number"
+F 5 "Yageo" H 3400 850 50  0001 C CNN "Manufacturer"
+F 6 "1" H 3400 850 50  0001 C CNN "Bin"
 	1    3400 850
 	1    0    0    -1
@@
 F 3 "~" H 1000 1000 50  0001 C CNN
 F 4 "GMK325BJ226MM-P" H 1000 1000 50  0001 C CNN "Part Number"
+F 5 "Taiyo Yuden" H 1000 1000 50  0001 C CNN "Manufacturer"
+F 6 "32" H 1000 1000 50  0001 C CNN "Bin"
 	1    1000 1000
 	1    0    0    -1

Commit message: Making some board modifications for the final revision
Parts:
- removed C2: 22uF, Capacitor_SMD:C_1210_3225Metric_Pad1.42x2.65mm_HandSolder, symbol Device:C
- removed C21, C6: 100nF, Capacitor_SMD:C_0603_1608Metric_Pad1.05x0.95mm_HandSolder, symbol Device:C
- removed C22, C4: 2.2uF, Capacitor_SMD:C_0603_1608Metric_Pad1.05x0.95mm_HandSolder, symbol Device:C
- removed C8: 1nF, Capacitor_SMD:C_0603_1608Metric_Pad1.05x0.95mm_HandSolder, symbol Device:C
- removed U1: DPS1133FIA-13, Snack Machine:DPS1133FIA-13, symbol Snack_Machine:DPS1133FIA-13
- added Q4: MMBT3904, Snack Machine:SOT-23_Handsoldering_Lite, symbol Transistor_BJT:MMBT3904
- added Q5: P-CH 30V 3.8A, Snack Machine:SOT-23_Handsoldering_Lite, symbol Device:Q_PMOS_GSD
- added R40: 47k, Resistor_SMD:R_0603_1608Metric_Pad1.05x0.95mm_HandSolder, symbol Device:R
- added R41: 10k, Resistor_SMD:R_0603_1608Metric_Pad1.05x0.95mm_HandSolder, symbol Device:R
- R18: value 330k -> 1k; Bin 20 -> (none); Manufacturer Yageo -> (none); Part Number RC0603FR-07330KL -> (none)
- R23: value 270k -> 10k; Bin 21 -> (none); Manufacturer Yageo -> (none); Part Number RC0603FR-07270KL -> (none)
- R24: value 100k -> 10k; Bin 16 -> (none); Manufacturer Yageo -> (none); Part Number RC0603FR-07100KL -> (none)
- R31: value 1k -> 4.7k; Bin 1 -> (none); Manufacturer Yageo -> (none); Part Number RC0603FR-071KL -> (none)
Connections:
- net MOTOR_CURRENT is gone; now on an unnamed net: R24.1
- net MOTOR_FAULT is gone; now on net GND: R31.2
- net +24V: now also R23.1, R24.2, Q5.2 (S)
- net GND: now also R41.2; no longer R18.2, R23.2, R24.2
- net MOTORS_ENABLE: now also R18.2
- net at D15.2 (A), U4.9 (VCC): now also Q5.3 (D), R40.1
- net at R18.1: now also Q4.1 (B)
- net +5V: no longer names the net of R31.1
- net +5V: now also Q4.2 (E)
- new net: Q4.3 (C), Q5.1 (G), R23.2
- new net MOTOR_SENSE: R40.2, R41.1
Other:
- note removed: "10 uA / A\n1 V/A with 100k"
- moved on the sheet: D15, U4

Commit message: Committing changes to the circuit board
Parts:
- R18: Bin (none) -> 1; Manufacturer (none) -> Yageo; Part Number (none) -> RC0603FR-071KL
- R23, R24, R41: Bin (none) -> 10; Manufacturer (none) -> Yageo; Part Number (none) -> RC0603FR-0710KL
- R31: Bin (none) -> 5; Manufacturer (none) -> Yageo; Part Number (none) -> RC0603FR-074K7L
- R40: Bin (none) -> 36; Manufacturer (none) -> Yageo; Part Number (none) -> RC0603FR-0747KL
Changed lines of the file:
@@
 F 2 "Resistor_SMD:R_0603_1608Metric_Pad1.05x0.95mm_HandSolder" V 1430 1950 50  0001 C CNN
 F 3 "~" H 1500 1950 50  0001 C CNN
+F 4 "Yageo" V 1500 1950 50  0001 C CNN "Manufacturer"
+F 5 "RC0603FR-071KL" V 1500 1950 50  0001 C CNN "Part Number"
+F 6 "1" V 1500 1950 50  0001 C CNN "Bin"
 	1    1500 1950
 	0    1    1    0
@@
 F 2 "Resistor_SMD:R_0603_1608Metric_Pad1.05x0.95mm_HandSolder" V 1980 2400 50  0001 C CNN
 F 3 "~" H 2050 2400 50  0001 C CNN
+F 4 "Yageo" H 2050 2400 50  0001 C CNN "Manufacturer"
+F 5 "RC0603FR-074K7L" H 2050 2400 50  0001 C CNN "Part Number"
+F 6 "5" H 2050 2400 50  0001 C CNN "Bin"
 	1    2050 2400
 	1    0    0    -1
@@
 F 2 "Resistor_SMD:R_0603_1608Metric_Pad1.05x0.95mm_HandSolder" V 1530 1450 50  0001 C CNN
 F 3 "~" H 1600 1450 50  0001 C CNN
+F 4 "RC0603FR-0710KL" H 1600 1450 50  0001 C CNN "Part Number"
+F 5 "Yageo" H 1600 1450 50  0001 C CNN "Manufacturer"
+F 6 "10" H 1600 1450 50  0001 C CNN "Bin"
 	1    1600 1450
 	1    0    0    -1
@@
 F 2 "Resistor_SMD:R_0603_1608Metric_Pad1.05x0.95mm_HandSolder" V 1980 850 50  0001 C CNN
 F 3 "~" H 2050 850 50  0001 C CNN
+F 4 "Yageo" V 2050 850 50  0001 C CNN "Manufacturer"
+F 5 "RC0603FR-0710KL" V 2050 850 50  0001 C CNN "Part Number"
+F 6 "10" V 2050 850 50  0001 C CNN "Bin"
 	1    2050 850
 	0    1    1    0
@@
 F 2 "Resistor_SMD:R_0603_1608Metric_Pad1.05x0.95mm_HandSolder" V 2830 1000 50  0001 C CNN
 F 3 "~" H 2900 1000 50  0001 C CNN
+F 4 "36" H 2900 1000 50  0001 C CNN "Bin"
+F 5 "Yageo" H 2900 1000 50  0001 C CNN "Manufacturer"
+F 6 "RC0603FR-0747KL" H 2900 1000 50  0001 C CNN "Part Number"
 	1    2900 1000
 	1    0    0    -1
@@
 F 2 "Resistor_SMD:R_0603_1608Metric_Pad1.05x0.95mm_HandSolder" V 2830 1500 50  0001 C CNN
 F 3 "~" H 2900 1500 50  0001 C CNN
+F 4 "RC0603FR-0710KL" H 2900 1500 50  0001 C CNN "Part Number"
+F 5 "Yageo" H 2900 1500 50  0001 C CNN "Manufacturer"
+F 6 "10" H 2900 1500 50  0001 C CNN "Bin"
 	1    2900 1500
 	1    0    0    -1

Commit message: current KiCad progress
Parts:
- added J8: Column Screw Terminal, TerminalBlock_Phoenix:TerminalBlock_Phoenix_PT-1,5-8-5.0-H_1x08_P5.00mm_Horizontal, symbol Connector:Screw_Terminal_01x08
- added J9: Row Screw Terminal, TerminalBlock_Phoenix:TerminalBlock_Phoenix_PT-1,5-8-5.0-H_1x08_P5.00mm_Horizontal, symbol Connector:Screw_Terminal_01x08
Connections:
- net col_1_ctrl renamed C1_MOTOR_CTRL
- net col_1_motor renamed c1_motor
- net c1_motor: now also J8.1 (Pin_1)
- net col_2_ctrl renamed C2_MOTOR_CTRL
- net col_2_motor renamed c2_motor
- net c2_motor: now also J8.2 (Pin_2)
- net col_3_ctrl renamed C3_MOTOR_CTRL
- net col_3_motor renamed c3_motor
- net c3_motor: now also J8.3 (Pin_3)
- net col_4_ctrl renamed C4_MOTOR_CTRL
- net col_4_motor renamed c4_motor
- net c4_motor: now also J8.4 (Pin_4)
- net col_5_ctrl renamed C5_MOTOR_CTRL
- net col_5_motor renamed c5_motor
- net c5_motor: now also J8.5 (Pin_5)
- net col_6_ctrl renamed C6_MOTOR_CTRL
- net col_6_motor renamed c6_motor
- net c6_motor: now also J8.6 (Pin_6)
- net col_7_ctrl renamed C7_MOTOR_CTRL
- net col_7_motor renamed c7_motor
- net c7_motor: now also J8.7 (Pin_7)
- net col_8_ctrl renamed C8_MOTOR_CTRL
- net col_8_motor renamed c8_motor
- net c8_motor: now also J8.8 (Pin_8)
- net row_a_ctrl renamed R1_MOTOR_CTRL
- net row_a_motor: no longer names the net of U4.18 (O1)
- net row_a_motor: now also J9.1 (Pin_1)
- net row_b_ctrl renamed R2_MOTOR_CTRL
- net row_b_motor: no longer names the net of U4.17 (O2)
- net row_b_motor: now also J9.2 (Pin_2)
- net row_c_ctrl renamed R3_MOTOR_CTRL
- net row_c_motor: no longer names the net of U4.16 (O3)
- net row_c_motor: now also J9.3 (Pin_3)
- net row_d_ctrl renamed R4_MOTOR_CTRL
- net row_d_motor: no longer names the net of U4.15 (O4)
- net row_d_motor: now also J9.4 (Pin_4)
- net row_e_ctrl renamed R5_MOTOR_CTRL
- net row_e_motor: no longer names the net of U4.14 (O5)
- net row_e_motor: now also J9.5 (Pin_5)
- net row_f_ctrl renamed R6_MOTOR_CTRL
- net row_f_motor: no longer names the net of U4.13 (O6)
- net row_f_motor: now also J9.6 (Pin_6)
- net row_g_ctrl renamed R7_MOTOR_CTRL
- net row_g_motor: no longer names the net of U4.12 (O7)
- net row_g_motor: now also J9.7 (Pin_7)
- net row_h_ctrl renamed R8_MOTOR_CTRL
- net row_h_motor: no longer names the net of U4.11 (O8)
- net row_h_motor: now also J9.8 (Pin_8)
Other:
- moved on the sheet: D11, D12, D13, D14, R17, R19, R2, R20, R21, R22, R8, R9
