File: KiCad/Huzzah32.sch (KiCad schematic (older format))
At the start: 6 parts

Commit message: Fixing ERC rules
Parts:
- gave numbers to parts that had none: 6
Changed lines of the file:
@@
 P 5050 2900
 AR Path="/5DE46DB4" Ref="U?"  Part="1"
-AR Path="/5DE1B8F8/5DE46DB4" Ref="U?"  Part="1"
-F 0 "U?" H 5050 3825 50  0000 C CNN
+AR Path="/5DE1B8F8/5DE46DB4" Ref="U5"  Part="1"
+F 0 "U5" H 5050 3825 50  0000 C CNN
 F 1 "Huzzah32" H 5050 3734 50  0000 C CNN
 F 2 "Snack Machine:HUZZAH32" H 4600 2050 50  0001 C CNN
@@
 AR Path="/5BCD883C/5DE46DBA" Ref="#PWR?"  Part="1"
 AR Path="/5DE46DBA" Ref="#PWR?"  Part="1"
-AR Path="/5DE1B8F8/5DE46DBA" Ref="#PWR?"  Part="1"
-F 0 "#PWR?" H 4300 1950 50  0001 C CNN
+AR Path="/5DE1B8F8/5DE46DBA" Ref="#PWR0138"  Part="1"
+F 0 "#PWR0138" H 4300 1950 50  0001 C CNN
 F 1 "+5V" H 4315 2273 50  0000 C CNN
 F 2 "" H 4300 2100 50  0001 C CNN
@@
 P 5900 2600
 AR Path="/5DE46DC0" Ref="#PWR?"  Part="1"
-AR Path="/5DE1B8F8/5DE46DC0" Ref="#PWR?"  Part="1"
-F 0 "#PWR?" H 5900 2350 50  0001 C CNN
+AR Path="/5DE1B8F8/5DE46DC0" Ref="#PWR0139"  Part="1"
+F 0 "#PWR0139" H 5900 2350 50  0001 C CNN
 F 1 "GND" H 5900 2450 50  0000 C CNN
 F 2 "" H 5900 2600 50  0001 C CNN
@@
 P 5800 2100
 AR Path="/5DE46DCA" Ref="#PWR?"  Part="1"
-AR Path="/5DE1B8F8/5DE46DCA" Ref="#PWR?"  Part="1"
-F 0 "#PWR?" H 5800 1950 50  0001 C CNN
+AR Path="/5DE1B8F8/5DE46DCA" Ref="#PWR0140"  Part="1"
+F 0 "#PWR0140" H 5800 1950 50  0001 C CNN
 F 1 "+3.3V" H 5815 2273 50  0000 C CNN
 F 2 "" H 5800 2100 50  0001 C CNN
@@
 	5700 2500 5900 2500
 $Comp
-L Logic_LevelTranslator:SN74LVC1T45DBV U?
+L Logic_LevelTranslator:SN74LVC1T45DBV U7
 U 1 1 5DE48758
 P 7800 2800
-F 0 "U?" H 8150 2650 50  0000 L CNN
+F 0 "U7" H 8150 2650 50  0000 L CNN
 F 1 "SN74LVC1T45DBV" H 8150 2550 50  0000 L CNN
 F 2 "Package_TO_SOT_SMD:SOT-23-6" H 7800 2350 50  0001 C CNN
@@
 	6300 2800 7400 2800
 $Comp
-L power:+5V #PWR?
+L power:+5V #PWR0141
 U 1 1 5DE4B549
 P 7700 2400
-F 0 "#PWR?" H 7700 2250 50  0001 C CNN
+F 0 "#PWR0141" H 7700 2250 50  0001 C CNN
 F 1 "+5V" H 7715 2573 50  0000 C CNN
 F 2 "" H 7700 2400 50  0001 C CNN
@@
 $EndComp
 $Comp
-L power:+3.3V #PWR?
+L power:+3.3V #PWR0142
 U 1 1 5DE4BB78
 P 7900 2400
-F 0 "#PWR?" H 7900 2250 50  0001 C CNN
+F 0 "#PWR0142" H 7900 2250 50  0001 C CNN
 F 1 "+3.3V" H 7915 2573 50  0000 C CNN
 F 2 "" H 7900 2400 50  0001 C CNN
@@
 HUZZAH_RX
 $Comp
-L power:GND #PWR?
+L power:GND #PWR0143
 U 1 1 5DE4C602
 P 7800 3200
-F 0 "#PWR?" H 7800 2950 50  0001 C CNN
+F 0 "#PWR0143" H 7800 2950 50  0001 C CNN
 F 1 "GND" H 7805 3027 50  0000 C CNN
 F 2 "" H 7800 3200 50  0001 C CNN
@@
 $EndComp
 $Comp
-L power:+5V #PWR?
+L power:+5V #PWR0144
 U 1 1 5DE4EE17
 P 7700 3650
-F 0 "#PWR?" H 7700 3500 50  0001 C CNN
+F 0 "#PWR0144" H 7700 3500 50  0001 C CNN
 F 1 "+5V" H 7715 3823 50  0000 C CNN
 F 2 "" H 7700 3650 50  0001 C CNN
@@
 $EndComp
 $Comp
-L power:+3.3V #PWR?
+L power:+3.3V #PWR0145
 U 1 1 5DE4EE1D
 P 7900 3650
-F 0 "#PWR?" H 7900 3500 50  0001 C CNN
+F 0 "#PWR0145" H 7900 3500 50  0001 C CNN
 F 1 "+3.3V" H 7915 3823 50  0000 C CNN
 F 2 "" H 7900 3650 50  0001 C CNN
@@
 $EndComp
 $Comp
-L power:GND #PWR?
+L power:GND #PWR0146
 U 1 1 5DE4EE24
 P 7800 4450
-F 0 "#PWR?" H 7800 4200 50  0001 C CNN
+F 0 "#PWR0146" H 7800 4200 50  0001 C CNN
 F 1 "GND" H 7805 4277 50  0000 C CNN
 F 2 "" H 7800 4450 50  0001 C CNN
@@
 HUZZAH_TX
 $Comp
-L power:GND #PWR?
+L power:GND #PWR0147
 U 1 1 5DE4FCE2
 P 7400 3000
-F 0 "#PWR?" H 7400 2750 50  0001 C CNN
+F 0 "#PWR0147" H 7400 2750 50  0001 C CNN
 F 1 "GND" H 7405 2827 50  0000 C CNN
 F 2 "" H 7400 3000 50  0001 C CNN
@@
 $EndComp
 $Comp
-L power:GND #PWR?
+L power:GND #PWR0148
 U 1 1 5DE515C6
 P 8200 4250
-F 0 "#PWR?" H 8200 4000 50  0001 C CNN
+F 0 "#PWR0148" H 8200 4000 50  0001 C CNN
 F 1 "GND" H 8205 4077 50  0000 C CNN
 F 2 "" H 8200 4250 50  0001 C CNN
@@
 $EndComp
 $Comp
-L Logic_LevelTranslator:SN74LVC1T45DBV U?
+L Logic_LevelTranslator:SN74LVC1T45DBV U8
 U 1 1 5DE4EE10
 P 7800 4050
-F 0 "U?" H 8150 3900 50  0000 L CNN
+F 0 "U8" H 8150 3900 50  0000 L CNN
 F 1 "SN74LVC1T45DBV" H 8150 3800 50  0000 L CNN
 F 2 "Package_TO_SOT_SMD:SOT-23-6" H 7800 3600 50  0001 C CNN
@@
 AR Path="/5BA75957/5DE58D00" Ref="Q?"  Part="1"
 AR Path="/5DE58D00" Ref="Q?"  Part="1"
-AR Path="/5DE1B8F8/5DE58D00" Ref="Q?"  Part="1"
-F 0 "Q?" H 7041 1346 50  0000 L CNN
+AR Path="/5DE1B8F8/5DE58D00" Ref="Q2"  Part="1"
+F 0 "Q2" H 7041 1346 50  0000 L CNN
 F 1 "MMBT3904" H 7041 1255 50  0000 L CNN
 F 2 "Snack Machine:SOT-23_Handsoldering_Lite" H 7050 1225 50  0001 L CIN
@@
 $EndComp
 $Comp
-L Device:R R?
+L Device:R R28
 U 1 1 5DE58D08
 P 7550 1550
-F 0 "R?" H 7400 1600 50  0000 C CNN
+F 0 "R28" H 7400 1600 50  0000 C CNN
 F 1 "4.7k" H 7400 1500 50  0000 C CNN
 F 2 "Resistor_SMD:R_0603_1608Metric_Pad1.05x0.95mm_HandSolder" V 7480 1550 50  0001 C CNN
@@
 $EndComp
 $Comp
-L Device:R R?
+L Device:R R27
 U 1 1 5DE58D10
 P 7300 1300
-F 0 "R?" V 7200 1300 50  0000 C CNN
+F 0 "R27" V 7200 1300 50  0000 C CNN
 F 1 "4.7k" V 7400 1300 50  0000 C CNN
 F 2 "Resistor_SMD:R_0603_1608Metric_Pad1.05x0.95mm_HandSolder" V 7230 1300 50  0001 C CNN
@@
 $EndComp
 $Comp
-L power:GND #PWR?
+L power:GND #PWR0149
 U 1 1 5DE58D16
 P 7550 1800
-F 0 "#PWR?" H 7550 1550 50  0001 C CNN
+F 0 "#PWR0149" H 7550 1550 50  0001 C CNN
 F 1 "GND" H 7600 1650 50  0000 R CNN
 F 2 "" H 7550 1800 50  0001 C CNN
@@
 $EndComp
 $Comp
-L power:GND #PWR?
+L power:GND #PWR0150
 U 1 1 5DE58D1C
 P 6750 1600
-F 0 "#PWR?" H 6750 1350 50  0001 C CNN
+F 0 "#PWR0150" H 6750 1350 50  0001 C CNN
 F 1 "GND" H 6800 1450 50  0000 R CNN
 F 2 "" H 6750 1600 50  0001 C CNN
@@
 Text HLabel 7550 1300 2    50   Input ~ 0
 RESET
+$Comp
+L power:+3.3V #PWR?
+U 1 1 5DD23E2B
+P 5150 1500
+F 0 "#PWR?" H 5150 1350 50  0001 C CNN
+F 1 "+3.3V" H 5165 1673 50  0000 C CNN
+F 2 "" H 5150 1500 50  0001 C CNN
+F 3 "" H 5150 1500 50  0001 C CNN
+	1    5150 1500
+	1    0    0    -1
+$EndComp
+$Comp
+L power:PWR_FLAG #FLG?
+U 1 1 5DD24501
+P 5150 1500
+F 0 "#FLG?" H 5150 1575 50  0001 C CNN
+F 1 "PWR_FLAG" H 5150 1673 50  0000 C CNN
+F 2 "" H 5150 1500 50  0001 C CNN
+F 3 "~" H 5150 1500 50  0001 C CNN
+	1    5150 1500
+	-1   0    0    1
+$EndComp
 $EndSCHEMATC
