File: KiCad/Huzzah32.sch (KiCad schematic (older format))
At the start: 6 parts, among them Q2 MMBT3904, U5 Huzzah32, U7 SN74LVC1T45DBV, U8 SN74LVC1T45DBV

Commit message: Current WIP for board layout
Connections:
- net HUZZAH_TX: no longer U5.14 (TX), U8.4 (B)
- new net: U5.14 (TX), U8.4 (B)
Changed lines of the file:
@@
 Wire Wire Line
 	5700 3600 6300 3600
-Text Label 5750 3600 0    50   ~ 0
-HUZZAH_TX
 $Comp
 L power:+3.3V #PWR?

Commit message: Rotated serial ports around to make routing easier
Connections:
- net HUZZAH_RX renamed RX_HUZZAH
- net HUZZAH_TX renamed TX_HUZZAH
Changed lines of the file:
@@
 $EndComp
 Text HLabel 8200 2800 2    50   Input ~ 0
-HUZZAH_RX
+RX_HUZZAH
 $Comp
 L power:GND #PWR0143
@@
 Wire Wire Line
 	6300 4050 7400 4050
-Text HLabel 8200 4050 2    50   Input ~ 0
-HUZZAH_TX
+Text HLabel 8200 4050 2    50   Output ~ 0
+TX_HUZZAH
 $Comp
 L power:GND #PWR0147

Commit message: Added part number, manufacturer, and personal bin numbers
Parts:
- Q2: Bin (none) -> 12
- R27, R28: Bin (none) -> 5
- U7, U8: Bin (none) -> 31; Manufacturer (none) -> Texas Instruments; Part Number (none) -> SN74LVC1T45DBV
Changed lines of the file:
@@
 F 2 "Package_TO_SOT_SMD:SOT-23-6" H 7800 2350 50  0001 C CNN
 F 3 "http://www.ti.com/lit/ds/symlink/sn74lvc1t45.pdf" H 6900 2150 50  0001 C CNN
+F 4 "SN74LVC1T45DBV" H 7800 2800 50  0001 C CNN "Part Number"
+F 5 "Texas Instruments" H 7800 2800 50  0001 C CNN "Manufacturer"
+F 6 "31" H 7800 2800 50  0001 C CNN "Bin"
 	1    7800 2800
 	1    0    0    -1
@@
 F 2 "Package_TO_SOT_SMD:SOT-23-6" H 7800 3600 50  0001 C CNN
 F 3 "http://www.ti.com/lit/ds/symlink/sn74lvc1t45.pdf" H 6900 3400 50  0001 C CNN
+F 4 "SN74LVC1T45DBV" H 7800 4050 50  0001 C CNN "Part Number"
+F 5 "Texas Instruments" H 7800 4050 50  0001 C CNN "Manufacturer"
+F 6 "31" H 7800 4050 50  0001 C CNN "Bin"
 	1    7800 4050
 	-1   0    0    -1
@@
 F 2 "Snack Machine:SOT-23_Handsoldering_Lite" H 7050 1225 50  0001 L CIN
 F 3 "https://www.fairchildsemi.com/datasheets/2N/2N3904.pdf" H 6850 1300 50  0001 L CNN
-F 4 "MMBT3904-TP" H 6850 1300 50  0001 C CNN "Part Number"
-F 5 "MCC" H 6850 1300 50  0001 C CNN "Manufacturer"
+F 4 "MCC" H 6850 1300 50  0001 C CNN "Manufacturer"
+F 5 "MMBT3904-TP" H 6850 1300 50  0001 C CNN "Part Number"
+F 6 "12" H 6850 1300 50  0001 C CNN "Bin"
 	1    6850 1300
 	-1   0    0    -1
@@
 F 4 "RC0603FR-074K7L" H 7550 1550 50  0001 C CNN "Part Number"
 F 5 "Yageo" H 7550 1550 50  0001 C CNN "Manufacturer"
+F 6 "5" H 7550 1550 50  0001 C CNN "Bin"
 	1    7550 1550
 	-1   0    0    -1
@@
 F 4 "RC0603FR-074K7L" V 7300 1300 50  0001 C CNN "Part Number"
 F 5 "Yageo" V 7300 1300 50  0001 C CNN "Manufacturer"
+F 6 "5" V 7300 1300 50  0001 C CNN "Bin"
 	1    7300 1300
 	0    -1   1    0

Commit message: Updating board to remove EXP1/EXP2
Connections:
- net RX_HUZZAH renamed HUZZAH_RX
- net TX_HUZZAH renamed HUZZAH_TX
Changed lines of the file:
@@
 $EndComp
 Text HLabel 8200 2800 2    50   Input ~ 0
-RX_HUZZAH
+HUZZAH_RX
 $Comp
 L power:GND #PWR0143
@@
 	6300 4050 7400 4050
 Text HLabel 8200 4050 2    50   Output ~ 0
-TX_HUZZAH
+HUZZAH_TX
 $Comp
 L power:GND #PWR0147
