File: KiCad/Snack Machine.kicad_pcb (KiCad board)
At the start: 2 copper layers, 107.5 x 100 mm, 286 parts, among them J1 MDB, J10 Row Screw Terminal, J11 Column Screw Terminal, J12 Display Serial Header, J13 RFID_CONNECTOR, J14 Large Display Header, J16 USB_B_Micro, J17 AVR-ISP-6, J18 Conn_02x02_Odd_Even, J2 Power Screw Terminal, J3 RFID Serial Connector, J4 RFID Led Connector, J5 MDB, J6 Conn_01x02, J7 LCD EXP1, J8 LCD EXP2, J9 AVR-ISP-6, Q1 P-CH 30V 3.8A, Q10 MMBT3904, Q11 P-CH 30V 3.8A, Q12 P-CH 30V 3.8A, Q13 P-CH 30V 3.8A, Q14 P-CH 30V 3.8A, Q15 MMBT3904, Q16 MMBT3904, Q17 MMBT3904, Q18 MMBT3904, Q19 Q_NMOS_SGD, Q2 Q_NMOS_SGD, Q20 Q_NMOS_SGD, Q21 Q_NMOS_SGD, Q22 Q_NMOS_SGD, Q23 Q_NMOS_SGD, Q24 Q_NMOS_SGD, Q25 Q_NMOS_SGD, Q26 MMBT3904, Q27 BSS138, Q28 BSS138, Q3 P-CH 30V 3.8A, Q4 P-CH 30V 3.8A, Q5 P-CH 30V 3.8A, Q6 P-CH 30V 3.8A, Q7 MMBT3904, Q8 MMBT3904, Q9 MMBT3904, SW1 SW_SPST, U2 MEZD71202A-G, U3 ATmega2560-16AU, U4 INA180B3, U5 INA219, U6 ATmega16U2-MU, U7 Huzzah32, Y1 16MHz, Y2 16MHz

Commit message: fixed a few small issues
Parts:
- added TP94: TestPoint, Snack Machine:TestPoint_THTPad_D0.8mm_Drill0.4mm, F.Cu at (132.2, 118.3)
- C21, C22: value 0.1uF -> 100nF
- Q27, Q28: footprint Package_TO_SOT_SMD:SOT-23 -> Snack Machine:SOT-23_Handsoldering_Lite
- R20, R22, R24, R25, R26, R27, R29, R30, R35, R36, R37, R39, R40, R41, R42, R43, R7: value 1K -> 1k
- moved TP93 5.89 mm to (111.4, 84.6)
- moved C24 4.86 mm to (113.1, 87.9), turned to 270 degrees
- moved TP25 4.70 mm to (127.5, 118.6)
- moved C26 2.49 mm to (111.4, 87.9), turned to 270 degrees
- moved R91 2.00 mm to (155.5, 91.8)
- moved R93 2.00 mm to (162.9, 91.8)
- moved F2 1.06 mm to (107.3, 89.2)
- moved Q27 0.90 mm to (156.4, 88.0)
- moved Q28 0.90 mm to (163.8, 88.0)
- moved G*** 0.41 mm to (185.4, 118.6)
- moved G*** 0.40 mm to (185.0, 106.7)
- moved G*** 0.22 mm to (185.2, 92.4)
Routing:
- net /CS: track 0.00 -> 8.21 mm, vias 0 -> 1
- net /USB_Serial/USBVCC: track 45.8 -> 51.6 mm
- net GND: track 967.4 -> 962.7 mm
- net Net-(TP25-Pad1): track 6.22 -> 10.9 mm
- net /RFID_GREEN_LED: track 43.2 -> 39.5 mm
- net /RFID_DATA_1: track 35.3 -> 38.8 mm
- net +5V: track 473.4 -> 476.2 mm
- net Net-(Q27-Pad3): track 36.5 -> 34.0 mm
- net Net-(Q28-Pad3): track 41.1 -> 39.2 mm
- net /RFID_RED_LED: track 43.1 -> 41.7 mm
- net +3V3: track 27.1 -> 28.4 mm
- net /RFID_DATA_0: track 34.4 -> 35.5 mm
- net /USB_Serial/XVCC: track 5.72 -> 6.78 mm
- net /RFID_BEEP: track 39.9 -> 38.9 mm
- net /LCD_PB: track 75.5 -> 76.2 mm
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
Commit message: Current WIP for board layout
Parts:
- removed C17, C18, C19, C20, C7, C9: OPEN, Capacitor_SMD:C_0603_1608Metric_Pad1.05x0.95mm_HandSolder
- removed C28: 100nF, Capacitor_SMD:C_0603_1608Metric_Pad1.05x0.95mm_HandSolder
- removed C46, C47, C48, C49, C50, C51, C52, C53: 1uF 50V, Capacitor_SMD:C_0603_1608Metric_Pad1.05x0.95mm_HandSolder
- removed D7, D8: D_Schottky, Diode_SMD:D_SOD-323
- removed FB1: 600R@100MHz, Inductor_SMD:L_0603_1608Metric_Pad1.05x0.95mm_HandSolder
- removed G***: LOGO, Snack Machine:TGD-logo
- removed G***: LOGO, Snack Machine:denhac-logo
- removed G***: LOGO, Snack Machine:oshw-logo
- removed H1, H2, H3, H4: MountingHole_Pad, MountingHole:MountingHole_3.5mm_Pad
- removed J13: RFID_CONNECTOR, Connector_PinHeader_2.54mm:PinHeader_1x05_P2.54mm_Vertical
- removed J14: Large Display Header, Connector_PinSocket_2.54mm:PinSocket_2x15_P2.54mm_Vertical
- removed J16: USB_B_Micro, Snack Machine:Amphenol_10118193-0001LF
- removed J18: Conn_02x02_Odd_Even, Connector_PinHeader_2.54mm:PinHeader_2x02_P2.54mm_Vertical
- removed JP1, JP2: SolderJumper_2_Open, Jumper:SolderJumper-2_P1.3mm_Open_TrianglePad1.0x1.5mm
- removed Q10, Q15, Q16, Q17, Q18, Q26, Q7, Q8, Q9: MMBT3904, Snack Machine:SOT-23_Handsoldering_Lite
- removed Q11, Q12, Q13, Q14, Q4, Q5, Q6: P-CH 30V 3.8A, Snack Machine:TSOT-23_HandSoldering_Lite
- removed Q19, Q20, Q21, Q22, Q23, Q24, Q25: Q_NMOS_SGD, Snack Machine:TSOT-23_HandSoldering_Lite
- removed Q27, Q28: BSS138, Snack Machine:SOT-23_Handsoldering_Lite
- removed R11: 0R, Resistor_SMD:R_0603_1608Metric_Pad1.05x0.95mm_HandSolder
- removed R32, R34, R35, R36, R37, R39, R40, R41, R42, R43, R44, R45, R46, R47, R48, R49, R50, R51, R79, R80, R81, R82: 1k, Resistor_SMD:R_0603_1608Metric_Pad1.05x0.95mm_HandSolder
- removed R33, R52, R53, R54, R83, R84, R85, R86, R90, R91, R92, R93: 10k, Resistor_SMD:R_0603_1608Metric_Pad1.05x0.95mm_HandSolder
- removed R38: 0.1R 1%, Resistor_SMD:R_0805_2012Metric_Pad1.15x1.40mm_HandSolder
- removed R88, R89: 4.7k, Resistor_SMD:R_0603_1608Metric_Pad1.05x0.95mm_HandSolder
- removed TP1, TP10, TP11, TP12, TP13, TP14, TP15, TP16, TP17, TP18, TP19, TP2, TP20, TP21, TP22, TP23, TP24, TP25, TP26, TP27, TP28, TP29, TP3, TP30, TP31, TP32, TP33, TP34, TP35, TP36, TP37, TP38, TP39, TP4, TP40, TP41, TP42, TP43, TP44, TP45, TP46, TP47, TP48, TP49, TP5, TP50, TP51, TP52, TP53, TP54, TP55, TP56, TP57, TP58, TP59, TP6, TP60, TP61, TP62, TP63, TP64, TP65, TP66, TP67, TP68, TP69, TP7, TP70, TP71, TP72, TP73, TP74, TP75, TP76, TP77, TP78, TP79, TP8, TP80, TP81, TP82, TP83, TP84, TP85, TP86, TP87, TP88, TP89, TP9, TP90, TP91, TP92, TP93, TP94: TestPoint, Snack Machine:TestPoint_THTPad_D0.8mm_Drill0.4mm
- added C2: 22 uF, Capacitor_SMD:C_1210_3225Metric_Pad1.42x2.65mm_HandSolder, B.Cu at (120.8, 94.6)
- added C4: 2.2 uF, Capacitor_SMD:C_0603_1608Metric_Pad1.05x0.95mm_HandSolder, B.Cu at (116.2, 96.3)
- added C6: 100 nF, Capacitor_SMD:C_0603_1608Metric_Pad1.05x0.95mm_HandSolder, B.Cu at (123.8, 98.1)
- added C8: 1 nF, Capacitor_SMD:C_0603_1608Metric_Pad1.05x0.95mm_HandSolder, B.Cu at (118.8, 109.3)
- added D15: S1GTR, Diode_SMD:D_SMA_Handsoldering, B.Cu at (113.1, 99.8)
- added TH1: tooling_hole, Snack Machine:tooling_hole_2.55, F.Cu at (103.0, 43.0)
- added TH2: tooling_hole, Snack Machine:tooling_hole_2.55, F.Cu at (173.0, 43.0)
- added TH3: tooling_hole, Snack Machine:tooling_hole_2.55, F.Cu at (103.0, 143.0)
- added TH4: tooling_hole, Snack Machine:tooling_hole_2.55, F.Cu at (173.0, 143.0)
- added U1: DPS1133FIA-13, Snack Machine:DPS1133FIA-13, B.Cu at (118.0, 102.0)
- added U8: SN74LVC1T45DBV, Package_TO_SOT_SMD:SOT-23-6, B.Cu at (136.3, 62.8)
- C21: value 100nF -> 100 nF; moved to B.Cu
- C22: value 100nF -> 2.2 uF; moved to B.Cu
- C24, C26, C3, D2, F2, R12, R15, R16, R58, R7, RV1, RV2: moved to B.Cu
- C29: moved to F.Cu
- D1, D10, D3, D9: value 50V 2A -> Q_TRIAC_A1A2G; footprint Snack Machine:D_SMB_Handsoldering_Lite -> Package_TO_SOT_SMD:SOT-223-3_TabPin2
- D11, D12, D13, D14: value 50V 2A -> Q_TRIAC_A1A2G; footprint Snack Machine:D_SMB_Handsoldering_Lite -> Package_TO_SOT_SMD:SOT-223-3_TabPin2; moved to B.Cu
- J1: value MDB -> RFID_CONNECTOR; footprint Connector_Molex:Molex_Mini-Fit_Jr_5566-06A_2x03_P4.20mm_Vertical -> Connector_PinHeader_2.54mm:PinHeader_1x10_P2.54mm_Vertical
- J12: footprint Connector_PinSocket_2.54mm:PinSocket_2x05_P2.54mm_Vertical -> Snack Machine:PinHeader_2x05_P2.54mm_Vertical; moved to F.Cu
- J3: value RFID Serial Connector -> USB_C_Receptacle_USB2.0; footprint Connector_PinHeader_2.54mm:PinHeader_1x05_P2.54mm_Vertical -> Snack Machine:USB_C_Receptacle_HRO_TYPE-C-31-M-12; moved to B.Cu
- J4: value RFID Led Connector -> V2 Display Ribbon Cable; footprint Connector_PinHeader_2.54mm:PinHeader_1x03_P2.54mm_Vertical -> Snack Machine:FPC30
- J6: footprint Connector_JST:JST_XH_B02B-XH-A_1x02_P2.50mm_Vertical -> Connector_PinHeader_2.54mm:PinHeader_1x02_P2.54mm_Vertical
- J7, J8: footprint Connector_PinHeader_2.54mm:PinHeader_2x05_P2.54mm_Vertical -> Snack Machine:PinHeader_2x05_P2.54mm_Vertical
- Q2: value Q_NMOS_SGD -> MMBT3904; footprint Snack Machine:TSOT-23_HandSoldering_Lite -> Snack Machine:SOT-23_Handsoldering_Lite
- Q3: value P-CH 30V 3.8A -> MMBT3904; footprint Snack Machine:TSOT-23_HandSoldering_Lite -> Snack Machine:SOT-23_Handsoldering_Lite
- R1: value 0R -> 1k
- R17, R19, R20, R22: value 1k -> 1 k
- R18: value 1k -> 330 k; moved to B.Cu
- R2, R8, R9: value 0R -> 1 k
- R21: value 10k -> 1 k
- R23: value 0.1R 1% -> 270 k; footprint Resistor_SMD:R_0805_2012Metric_Pad1.15x1.40mm_HandSolder -> Resistor_SMD:R_0603_1608Metric_Pad1.05x0.95mm_HandSolder; moved to B.Cu
- R24: value 1k -> 100 k
- R25, R26: value 1k -> 5.1 k
- R27, R29, R30: value 1k -> 4.7k
- R28: value 10k -> 4.7k; moved to B.Cu
- R31: value 1k -> 1 k; moved to F.Cu
- U4: value INA180B3 -> TBD62783A; footprint Package_TO_SOT_SMD:SOT-23-5_HandSoldering -> Package_SO:SSOP-18_4.4x6.5mm_P0.65mm; moved to B.Cu
- U5: value INA219 -> Huzzah32; footprint Package_TO_SOT_SMD:TSOT-23-8_HandSoldering -> Snack Machine:HUZZAH32
- U7: value Huzzah32 -> SN74LVC1T45DBV; footprint Snack Machine:HUZZAH32 -> Package_TO_SOT_SMD:SOT-23-6; moved to B.Cu
- moved J2 102.4 mm to (106.0, 82.9), turned to 270 degrees
- moved Q3 100.3 mm to (203.9, 54.9)
- moved F1 98.0 mm to (115.0, 79.7), turned to 270 degrees
- moved R30 86.2 mm to (199.6, 57.4), turned to 270 degrees
- moved C30 85.8 mm to (155.9, 21.4), turned to 0 degrees
- moved R26 85.6 mm to (159.7, 50.9), turned to 180 degrees
- moved R25 85.2 mm to (165.3, 50.8)
- moved SW1 83.5 mm to (113.9, 44.7)
- moved R29 82.6 mm to (205.8, 69.3), turned to 180 degrees
- moved D4 81.8 mm to (149.3, 36.4), turned to 0 degrees
- moved J11 80.4 mm to (116.3, 140.3), turned to 0 degrees
- moved R12 80.3 mm to (119.4, 44.7), turned to 270 degrees
- moved R58 79.2 mm to (149.9, 42.1), turned to 0 degrees
- moved R7 78.7 mm to (115.6, 48.0)
- moved D2 78.7 mm to (117.1, 44.2), turned to 90 degrees
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Connections:
- C21 pad 1: +5V -> /MOTOR_CURRENT
- C22 pad 1: +5V -> Net-(C22-Pad1)
- C27 pad 2: /USB_Serial/USB_GND -> GND
- C3 pad 1: VCC -> +5V
- D1 pad 1: /MotorPower/row_a_motor -> GND
- D1 pad 2: GND -> /MotorPower/col_1_motor
- D10 pad 1: /MotorPower/row_d_motor -> GND
- D10 pad 2: GND -> /MotorPower/col_7_motor
- D11 pad 1: /MotorPower/row_e_motor -> GND
- D11 pad 2: GND -> /MotorPower/col_2_motor
- D12 pad 1: /MotorPower/row_f_motor -> GND
- D12 pad 2: GND -> /MotorPower/col_4_motor
- D13 pad 1: /MotorPower/row_g_motor -> GND
- D13 pad 2: GND -> /MotorPower/col_6_motor
- D14 pad 1: /MotorPower/row_h_motor -> GND
- D14 pad 2: GND -> /MotorPower/col_8_motor
- D3 pad 1: /MotorPower/row_b_motor -> GND
- D3 pad 2: GND -> /MotorPower/col_3_motor
- D9 pad 1: /MotorPower/row_c_motor -> GND
- D9 pad 2: GND -> /MotorPower/col_5_motor
- J1 pad 1: +24V -> +5V
- J1 pad 3: Net-(J1-Pad3) -> GND
- J1 pad 4: /RX_MDB -> /RFID_GREEN_LED
- J1 pad 5: Net-(J1-Pad5) -> /RFID_RED_LED
- J1 pad 6: GND -> /RFID_BEEP_CTRL
- J12 pad 1: VCC -> +5V
- J12 pad 10: Net-(J12-Pad10) -> (no net)
- J12 pad 2: Net-(J12-Pad2) -> (no net)
- J12 pad 3: /TX_DISPLAY -> /4D_Display/TX_DISPLAY
- J12 pad 4: Net-(J12-Pad4) -> (no net)
- J12 pad 5: /RX_DISPLAY -> /4D_Display/RX_DISPLAY
- J12 pad 6: Net-(J12-Pad6) -> (no net)
- J12 pad 8: Net-(J12-Pad8) -> (no net)
- J12 pad 9: Net-(J12-Pad9) -> /4D_Display/RESET
- J4 pad 1: /RFID_LED -> GND
- J4 pad 2: +5V -> (no net)
- J4 pad 3: GND -> (no net)
- J5 pad 3: Net-(J5-Pad3) -> (no net)
- J5 pad 5: Net-(J1-Pad5) -> Net-(J5-Pad5)
- J7 pad 1: /BEEPER -> /LCD_BEEP
- J7 pad 3: /LCD_SDA -> /LCD_EN
- J7 pad 5: /LCD_SCL -> /LCD_4
- J7 pad 6: Net-(J7-Pad6) -> /LCD_5
- J7 pad 7: Net-(J7-Pad7) -> /LCD_6
- J7 pad 8: Net-(J7-Pad8) -> /LCD_7
- J8 pad 1: Net-(J8-Pad1) -> /MISO
- J8 pad 10: Net-(J8-Pad10) -> (no net)
- J8 pad 2: Net-(J8-Pad2) -> /SCK
- J8 pad 4: Net-(J8-Pad4) -> /SD_CS
- J8 pad 6: Net-(J8-Pad6) -> /MOSI
- J8 pad 7: Net-(J8-Pad7) -> /SD_DET
- J8 pad 8: /LCD_PB -> /LCD_RESET
- J8 pad 9: GND -> (no net)
- Q1 pad 1: Net-(Q1-Pad1) -> /TX_MDB
- Q1 pad 3: Net-(J1-Pad5) -> Net-(J5-Pad5)
- Q2 pad 2: /MotorPower/motor_common_gnd -> GND
- Q2 pad 3: /MotorPower/col_1_motor -> Net-(Q2-Pad3)
- Q3 pad 2: +24V -> GND
- Q3 pad 3: /MotorPower/row_b_motor -> /4D_Display/RESET
- R1 pad 1: /SDA -> /RX_MDB
- R1 pad 2: /LCD_SDA -> +5V
- R13 pad 1: /TX_DISPLAY -> /4D_Display/TX_DISPLAY
- R13 pad 2: Net-(C19-Pad1) -> Net-(R13-Pad2)
- R14 pad 1: /RX_DISPLAY -> /4D_Display/RX_DISPLAY
- R14 pad 2: Net-(C17-Pad1) -> Net-(R14-Pad2)
- R17 pad 1: +5V -> /c7
- R17 pad 2: /SCL -> Net-(D10-Pad3)
- R18 pad 1: +5V -> Net-(R18-Pad1)
- R18 pad 2: /SDA -> GND
- R19 pad 1: Net-(Q7-Pad1) -> /c2
- R19 pad 2: /r1 -> Net-(D11-Pad3)
- R2 pad 1: /SCL -> /c1
- R2 pad 2: /LCD_SCL -> Net-(D1-Pad3)
- R20 pad 1: Net-(Q3-Pad1) -> /c4
- R20 pad 2: +24V -> Net-(D12-Pad3)
- R21 pad 1: /MotorPower/motor_common_gnd -> /c6
- R21 pad 2: Net-(Q2-Pad1) -> Net-(D13-Pad3)
- R22 pad 1: Net-(Q4-Pad1) -> /c8
- R22 pad 2: +24V -> Net-(D14-Pad3)
- R23 pad 1: GND -> Net-(R23-Pad1)
- R23 pad 2: /MotorPower/motor_common_gnd -> GND
- R24 pad 1: Net-(Q5-Pad1) -> /MOTOR_CURRENT
- R24 pad 2: +24V -> GND
- R25 pad 1: Net-(Q6-Pad1) -> Net-(J3-PadB5)
- R25 pad 2: Net-(Q7-Pad3) -> GND
- R26 pad 1: Net-(Q6-Pad1) -> Net-(J3-PadA5)
- R26 pad 2: +24V -> GND
- R27 pad 1: Net-(Q3-Pad1) -> Net-(Q2-Pad1)
- R27 pad 2: Net-(Q8-Pad3) -> /Huzzah32/RESET
- R28 pad 1: Net-(JP1-Pad2) -> /Huzzah32/RESET
- R29 pad 1: Net-(Q4-Pad1) -> /RESET_DISPLAY
- R29 pad 2: Net-(Q9-Pad3) -> GND
- R30 pad 1: Net-(Q5-Pad1) -> Net-(Q3-Pad1)
- R30 pad 2: Net-(Q10-Pad3) -> /RESET_DISPLAY
- R31 pad 1: Net-(Q8-Pad1) -> +5V
- R31 pad 2: /r2 -> /MOTOR_FAULT
- R4 pad 1: Net-(Q1-Pad1) -> /TX_MDB
- R5 pad 1: Net-(Q1-Pad1) -> /TX_MDB
- R5 pad 2: /TX_MDB -> Net-(R5-Pad2)
- R8 pad 1: /RFID_RX -> /c3
- R8 pad 2: Net-(C17-Pad1) -> Net-(D3-Pad3)
- R9 pad 1: /RFID_TX -> /c5
- R9 pad 2: Net-(C19-Pad1) -> Net-(D9-Pad3)
- RV1 pad 2: /USB_Serial/USB_SHIELD -> GND
- RV2 pad 2: /USB_Serial/USB_SHIELD -> GND
- U2 pad 3: VCC -> +5V
- U3 pad 1: Net-(TP27-Pad1) -> (no net)
- U3 pad 13: Net-(C9-Pad1) -> Net-(R5-Pad2)
- U3 pad 14: Net-(TP20-Pad1) -> (no net)
- U3 pad 15: Net-(TP21-Pad1) -> (no net)
- U3 pad 16: Net-(TP22-Pad1) -> (no net)
- U3 pad 17: Net-(TP23-Pad1) -> (no net)
- U3 pad 18: Net-(TP24-Pad1) -> (no net)
- U3 pad 19: /CS -> (no net)
- U3 pad 23: Net-(TP28-Pad1) -> /BTN_ENC
- U3 pad 24: /BEEPER -> /SD_DET
- U3 pad 25: /RFID_LED -> /DOOR_SW
- U3 pad 26: /RFID_BEEP -> (no net)
- U3 pad 27: Net-(TP25-Pad1) -> (no net)
- U3 pad 29: Net-(TP26-Pad1) -> /RFID_BEEP_CTRL
- U3 pad 4: Net-(TP40-Pad1) -> (no net)
- U3 pad 43: /SCL -> /MOTOR_FAULT
- U3 pad 44: /SDA -> /MOTORS_ENABLE
- U3 pad 45: Net-(C19-Pad1) -> Net-(R13-Pad2)
- U3 pad 46: Net-(C17-Pad1) -> Net-(R14-Pad2)
- U3 pad 47: Net-(TP36-Pad1) -> (no net)
- U3 pad 48: Net-(TP37-Pad1) -> (no net)
- U3 pad 49: Net-(TP38-Pad1) -> (no net)
- U3 pad 5: Net-(TP41-Pad1) -> (no net)
- U3 pad 50: Net-(TP39-Pad1) -> (no net)
- U3 pad 51: /LCD_CS -> /SD_CS
- U3 pad 63: Net-(Q27-Pad3) -> /Huzzah32/HUZZAH_TX
- U3 pad 64: Net-(Q28-Pad3) -> /Huzzah32/HUZZAH_RX
- U3 pad 65: /DOOR_SW -> /Huzzah32/RESET
- U3 pad 66: Net-(TP15-Pad1) -> (no net)
- U3 pad 67: Net-(TP16-Pad1) -> (no net)
- U3 pad 68: Net-(TP17-Pad1) -> (no net)
- U3 pad 69: Net-(TP18-Pad1) -> (no net)
- U3 pad 71: Net-(TP35-Pad1) -> (no net)
- U3 pad 72: Net-(TP34-Pad1) -> (no net)
- U3 pad 73: Net-(TP33-Pad1) -> (no net)
- U3 pad 74: Net-(TP32-Pad1) -> (no net)
- U3 pad 75: Net-(TP31-Pad1) -> (no net)
- U3 pad 76: Net-(TP30-Pad1) -> (no net)
- U3 pad 77: Net-(TP29-Pad1) -> (no net)
- U3 pad 79: Net-(TP19-Pad1) -> (no net)
- U3 pad 82: Net-(TP14-Pad1) -> /LCD_RESET
- U3 pad 83: Net-(TP13-Pad1) -> /LCD_7
- U3 pad 84: Net-(TP12-Pad1) -> /LCD_6
- U3 pad 85: Net-(TP11-Pad1) -> /LCD_5
- U3 pad 86: Net-(TP10-Pad1) -> /LCD_4
- U3 pad 87: Net-(TP9-Pad1) -> /LCD_EN
- U3 pad 88: /LCD_PB -> /LCD_CS
- U3 pad 89: /BTN_ENC -> /LCD_BEEP
- U3 pad 90: Net-(TP49-Pad1) -> (no net)
- U3 pad 91: Net-(TP48-Pad1) -> (no net)
- U3 pad 92: Net-(TP47-Pad1) -> (no net)
- U3 pad 93: Net-(TP46-Pad1) -> (no net)
- U3 pad 94: Net-(TP45-Pad1) -> (no net)
- U3 pad 95: Net-(TP44-Pad1) -> (no net)
- U3 pad 96: Net-(TP43-Pad1) -> (no net)
- U3 pad 97: Net-(TP42-Pad1) -> (no net)
- U4 pad 1: /MOTOR_CURRENT -> /r1
- U4 pad 2: GND -> /r2
- U4 pad 3: /MotorPower/motor_common_gnd -> /r3
- U4 pad 4: GND -> /r4
- U4 pad 5: +5V -> /r5
- U5 pad 1: Net-(JP1-Pad2) -> (no net)
- U5 pad 2: Net-(JP2-Pad2) -> (no net)
- U5 pad 3: /SDA -> +5V
- U5 pad 4: /SCL -> (no net)
- U5 pad 5: +5V -> (no net)
- U5 pad 6: GND -> (no net)
- U5 pad 7: GND -> (no net)
- U5 pad 8: /MotorPower/motor_common_gnd -> (no net)
- U6 pad 12: Net-(U6-Pad12) -> (no net)
- U6 pad 14: Net-(U6-Pad14) -> (no net)
- U6 pad 18: /USB_Serial/8PB4 -> (no net)
- U6 pad 19: /USB_Serial/8PB5 -> (no net)
- U6 pad 20: /USB_Serial/8PB6 -> (no net)
- U6 pad 21: /USB_Serial/8PB7 -> (no net)
- U6 pad 22: Net-(U6-Pad22) -> (no net)
- U6 pad 23: Net-(U6-Pad23) -> (no net)
- U6 pad 25: Net-(U6-Pad25) -> (no net)
- U6 pad 26: Net-(U6-Pad26) -> (no net)
- U6 pad 28: /USB_Serial/USB_GND -> GND
- U6 pad 5: Net-(U6-Pad5) -> (no net)
- U6 pad 6: Net-(U6-Pad6) -> (no net)
- U6 pad 7: Net-(U6-Pad7) -> (no net)
- U7 pad 1: Net-(U7-Pad1) -> +5V
- U7 pad 2: Net-(U7-Pad2) -> GND
- U7 pad 3: +5V -> Net-(U5-Pad15)
- U7 pad 4: Net-(U7-Pad4) -> /Huzzah32/HUZZAH_RX
- U7 pad 5: Net-(U7-Pad5) -> GND
- U7 pad 6: Net-(U7-Pad6) -> +3V3
Routing:
- net GND: track 962.7 -> 56.2 mm, vias 26 -> 11
- net +5V: track 476.2 -> 48.4 mm, vias 13 -> 2
- net /SCL: track 138.9 -> 0.00 mm, vias 4 -> 0
- net /SDA: track 136.2 -> 0.00 mm, vias 3 -> 0
- net /MotorPower/motor_common_gnd: track 85.8 -> 0.00 mm, vias 9 -> 0
- net VCC: track 85.8 -> 0.00 mm
- net /DOOR_SW: track 79.9 -> 0.00 mm, vias 1 -> 0
- net +24V: track 220.2 -> 143.9 mm, vias 8 -> 0
- net /LCD_PB: track 76.2 -> 0.00 mm, vias 2 -> 0
- net /LCD_CS: track 67.9 -> 0.00 mm, vias 2 -> 0
- net /RFID_TX: track 67.6 -> 0.00 mm
- net /BTN_EN1: track 63.4 -> 0.00 mm
- net /BTN_EN2: track 61.5 -> 0.00 mm
- net /BTN_ENC: track 60.2 -> 0.00 mm, vias 3 -> 0
- net /Huzzah32/RESET: track 0.00 -> 58.3 mm, vias 0 -> 1
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- added copper zone on F.Cu, net +5V
- removed copper zone on F.Cu, net GND
Other:
- board size 107.5 x 100 mm -> 76 x 106 mm
- net class High Amp: trace_width 0.8 -> 0.6
- rule pad_to_mask_clearance: 0.2 -> 0.0762
- rule solder_mask_min_width: 0.25 -> 0.1016
- rule via_min_drill: 0.3 -> 0.254
- rule via_min_size: 0.4 -> 0.508
- board text added: "16U2"
- board text added: "2560"
- board text removed: "Snack Machine Controller v1.0"

Commit message: Committing before changing schematic
Parts:
- C24, C26: moved to F.Cu
- C30, D4: moved to B.Cu
- moved C30 50.7 mm to (147.6, 71.4), turned to 90 degrees
- moved R14 43.1 mm to (162.5, 71.1), turned to 270 degrees
- moved R29 41.8 mm to (164.4, 63.5), turned to 90 degrees
- moved R13 40.9 mm to (164.5, 71.2), turned to 270 degrees
- moved Q3 40.3 mm to (163.8, 59.5), turned to 0 degrees
- moved R30 37.6 mm to (162.5, 63.6)
- moved C26 19.4 mm to (148.2, 57.0), turned to 180 degrees
- moved C24 19.4 mm to (148.2, 54.5), turned to 180 degrees
- moved RV2 15.5 mm to (155.0, 47.5), turned to 90 degrees
- moved C27 14.9 mm to (148.8, 56.2), turned to 180 degrees
- moved R3 10.7 mm to (159.6, 110.4)
- moved J6 10.7 mm to (164.0, 108.9)
- moved D4 7.52 mm to (147.6, 43.8), turned to 270 degrees
- moved R10 7.11 mm to (166.4, 127.8)
- moved RV1 5.90 mm to (164.9, 53.8)
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Routing:
- net +5V: track 48.4 -> 104.9 mm, vias 2 -> 4
- net /Huzzah32/HUZZAH_TX: track 52.5 -> 0.00 mm, vias 1 -> 0
- net /Huzzah32/HUZZAH_RX: track 48.0 -> 3.40 mm
- net /Huzzah32/RESET: track 58.3 -> 14.3 mm
- net /MISO: track 64.0 -> 27.6 mm, vias 2 -> 0
- net /SCK: track 59.0 -> 25.8 mm
- net Net-(R16-Pad2): track 0.00 -> 32.9 mm, vias 0 -> 1
- net /USB_Serial/~RESET2: track 0.00 -> 32.5 mm, vias 0 -> 2
- net /USB_Serial/SCK2: track 0.00 -> 30.2 mm, vias 0 -> 1
- net Net-(R15-Pad2): track 0.00 -> 29.9 mm, vias 0 -> 1
- net /LCD_RESET: track 0.00 -> 29.4 mm
- net /MOSI: track 56.8 -> 27.6 mm, vias 2 -> 0
- net /LCD_BEEP: track 0.00 -> 29.0 mm
- net /LCD_4: track 0.00 -> 28.8 mm, vias 0 -> 1
- net /LCD_EN: track 0.00 -> 28.7 mm, vias 0 -> 1
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