File: KiCad/USB_Serial.sch (KiCad schematic (older format))
At the start: 33 parts, among them J17 AVR-ISP-6, J18 Conn_02x02_Odd_Even, J3 USB_C_Receptacle_USB2.0, U6 ATmega16U2-MU, Y2 16MHz

Commit message: Current WIP for board layout
Parts:
- removed C28: 100nF, Capacitor_SMD:C_0603_1608Metric_Pad1.05x0.95mm_HandSolder, symbol Device:C
- removed D8: D_Schottky, Diode_SMD:D_SOD-323, symbol Device:D_Schottky
- removed J18: Conn_02x02_Odd_Even, Connector_PinHeader_2.54mm:PinHeader_2x02_P2.54mm_Vertical, symbol Connector_Generic:Conn_02x02_Odd_Even
- removed J3: USB_C_Receptacle_USB2.0, symbol Connector:USB_C_Receptacle_USB2.0
- removed TP92, TP93: TestPoint, Snack Machine:TestPoint_THTPad_D0.8mm_Drill0.4mm, symbol Connector:TestPoint
- added J3: USB_C_Receptacle_USB2.0, Snack Machine:USB_C_Receptacle_HRO_TYPE-C-31-M-12, symbol Snack_Machine:USB_C_Receptacle_USB2.0
- R25, R26: footprint (none) -> Resistor_SMD:R_0603_1608Metric_Pad1.05x0.95mm_HandSolder
Connections:
- net labels removed: 8PB4, 8PB5, 8PB6, 8PB7
- wire segments 109 -> 92
- no-connect marks 11 -> 15
Other:
- moved on the sheet: C29
Changed lines of the file:
@@
-$EndComp
-$Comp
-L Device:C C28
-U 1 1 5BC6BAD9
-P 6750 1150
-F 0 "C28" H 6865 1196 50  0000 L CNN
-F 1 "100nF" H 6865 1105 50  0000 L CNN
-F 2 "Capacitor_SMD:C_0603_1608Metric_Pad1.05x0.95mm_HandSolder" H 6788 1000 50  0001 C CNN
-F 3 "~" H 6750 1150 50  0001 C CNN
-F 4 "CC0603KRX7R9BB104" H 6750 1150 50  0001 C CNN "Part Number"
-F 5 "Yageo" H 6750 1150 50  0001 C CNN "Manufacturer"
-	1    6750 1150
-	1    0    0    -1
 $EndComp
 $Comp
@@
 L Device:C C29
 U 1 1 5BE8C422
-P 7200 1150
-F 0 "C29" H 7315 1196 50  0000 L CNN
-F 1 "1uF" H 7315 1105 50  0000 L CNN
-F 2 "Capacitor_SMD:C_0603_1608Metric_Pad1.05x0.95mm_HandSolder" H 7238 1000 50  0001 C CNN
-F 3 "~" H 7200 1150 50  0001 C CNN
-F 4 "C1608X7R1A105K080AC" H 7200 1150 50  0001 C CNN "Part Number"
-F 5 "TDK" H 7200 1150 50  0001 C CNN "Manufacturer"
-	1    7200 1150
-	1    0    0    -1
-$EndComp
-Wire Wire Line
-	7200 1000 6750 1000
-Connection ~ 6750 1000
-Wire Wire Line
-	7200 1300 6750 1300
-Connection ~ 6750 1300
+P 6750 1150
+F 0 "C29" H 6865 1196 50  0000 L CNN
+F 1 "1uF" H 6865 1105 50  0000 L CNN
+F 2 "Capacitor_SMD:C_0603_1608Metric_Pad1.05x0.95mm_HandSolder" H 6788 1000 50  0001 C CNN
+F 3 "~" H 6750 1150 50  0001 C CNN
+F 4 "C1608X7R1A105K080AC" H 6750 1150 50  0001 C CNN "Part Number"
+F 5 "TDK" H 6750 1150 50  0001 C CNN "Manufacturer"
+	1    6750 1150
+	1    0    0    -1
+$EndComp
 Wire Wire Line
 	5350 1450 5800 1450
@@
 Text Notes 9900 5300 2    50   ~ 0
 NOTE: This is the RESET\nline for the ATMEGA2560
-Wire Wire Line
-	7450 3550 7850 3550
-Wire Wire Line
-	7450 3450 7850 3450
-Wire Wire Line
-	7450 3350 7850 3350
-Wire Wire Line
-	7450 3250 7850 3250
-Text Label 7550 3250 0    50   ~ 0
-8PB4
-Text Label 7550 3350 0    50   ~ 0
-8PB5
-Text Label 7550 3450 0    50   ~ 0
-8PB6
-Text Label 7550 3550 0    50   ~ 0
-8PB7
-Wire Wire Line
-	8950 1200 9350 1200
-Wire Wire Line
-	8950 1100 9350 1100
-Wire Wire Line
-	8050 1200 8450 1200
-Wire Wire Line
-	8050 1100 8450 1100
-Text Label 8150 1100 0    50   ~ 0
-8PB4
-Text Label 8150 1200 0    50   ~ 0
-8PB5
-Text Label 9050 1100 0    50   ~ 0
-8PB6
-Text Label 9050 1200 0    50   ~ 0
-8PB7
-$Comp
-L Connector_Generic:Conn_02x02_Odd_Even J18
-U 1 1 5C0260BF
-P 8650 1100
-F 0 "J18" H 8700 1317 50  0000 C CNN
-F 1 "Conn_02x02_Odd_Even" H 8700 1226 50  0000 C CNN
-F 2 "Connector_PinHeader_2.54mm:PinHeader_2x02_P2.54mm_Vertical" H 8650 1100 50  0001 C CNN
-F 3 "~" H 8650 1100 50  0001 C CNN
-	1    8650 1100
-	1    0    0    -1
-$EndComp
 Text Label 7700 5050 0    50   ~ 0
 DTR
-Text Label 1650 1750 2    50   ~ 0
-USBVCC
-Wire Wire Line
-	1750 1750 1300 1750
-$Comp
-L power:+5V #PWR093
-U 1 1 5C4A9D62
-P 2200 1650
-F 0 "#PWR093" H 2200 1500 50  0001 C CNN
-F 1 "+5V" H 2215 1823 50  0000 C CNN
-F 2 "" H 2200 1650 50  0001 C CNN
-F 3 "" H 2200 1650 50  0001 C CNN
-	1    2200 1650
-	1    0    0    -1
-$EndComp
-Wire Wire Line
-	2200 1750 2200 1650
 Wire Wire Line
 	6750 2400 6750 2450
@@
 Wire Wire Line
 	4450 2650 4900 2650
-Wire Wire Line
-	2050 1750 2200 1750
-$Comp
-L Device:D_Schottky D8
-U 1 1 5C21EC9A
-P 1900 1750
-F 0 "D8" H 1900 1534 50  0000 C CNN
-F 1 "D_Schottky" H 1900 1625 50  0000 C CNN
-F 2 "Diode_SMD:D_SOD-323" H 1900 1750 50  0001 C CNN
-F 3 "~" H 1900 1750 50  0001 C CNN
-F 4 "Toshiba Semiconductor and Storage" H 1900 1750 50  0001 C CNN "Manufacturer"
-F 5 "CUS08F30,H3F" H 1900 1750 50  0001 C CNN "Part Number"
-	1    1900 1750
-	-1   0    0    1
-$EndComp
 Text Label 5550 3450 0    50   ~ 0
 MICRO_D+
@@
 Text Label 7450 4650 0    50   ~ 0
 MICRO_RX
-Text Label 2650 1400 0    50   ~ 0
-USBVCC
-Wire Wire Line
-	2600 1400 3050 1400
-$Comp
-L Connector:TestPoint TP93
-U 1 1 5C3B0CCE
-P 3150 1500
-AR Path="/5BCD883C/5C3B0CCE" Ref="TP93"  Part="1"
-AR Path="/5C3B0CCE" Ref="TP?"  Part="1"
-F 0 "TP93" V 3100 1450 50  0000 L CNN
-F 1 "TestPoint" V 3100 1700 50  0000 L CNN
-F 2 "Snack Machine:TestPoint_THTPad_D0.8mm_Drill0.4mm" H 3350 1500 50  0001 C CNN
-F 3 "~" H 3350 1500 50  0001 C CNN
-	1    3150 1500
-	0    1    1    0
-$EndComp
-$Comp
-L Connector:TestPoint TP92
-U 1 1 5C3B7E84
-P 3150 1400
-AR Path="/5BCD883C/5C3B7E84" Ref="TP92"  Part="1"
-AR Path="/5C3B7E84" Ref="TP?"  Part="1"
-F 0 "TP92" V 3100 1350 50  0000 L CNN
-F 1 "TestPoint" V 3100 1600 50  0000 L CNN
-F 2 "Snack Machine:TestPoint_THTPad_D0.8mm_Drill0.4mm" H 3350 1400 50  0001 C CNN
-F 3 "~" H 3350 1400 50  0001 C CNN
-	1    3150 1400
-	0    1    1    0
-$EndComp
-Wire Wire Line
-	3050 1400 3050 1500
-Wire Wire Line
-	3050 1500 3150 1500
-Connection ~ 3050 1400
-Wire Wire Line
-	3050 1400 3150 1400
-$Comp
-L Connector:USB_C_Receptacle_USB2.0 J3
-U 1 1 5DCD228D
-P 1050 3000
-F 0 "J3" H 1157 3867 50  0000 C CNN
-F 1 "USB_C_Receptacle_USB2.0" H 1157 3776 50  0000 C CNN
-F 2 "" H 1200 3000 50  0001 C CNN
-F 3 "https://www.usb.org/sites/default/files/documents/usb_type-c.zip" H 1200 3000 50  0001 C CNN
-	1    1050 3000
-	1    0    0    -1
-$EndComp
 Wire Wire Line
 	1650 2400 2050 2400
@@
 F 0 "R26" H 3220 2796 50  0000 L CNN
 F 1 "5.1 k" H 3220 2705 50  0000 L CNN
-F 2 "" V 3080 2750 50  0001 C CNN
+F 2 "Resistor_SMD:R_0603_1608Metric_Pad1.05x0.95mm_HandSolder" V 3080 2750 50  0001 C CNN
 F 3 "~" H 3150 2750 50  0001 C CNN
 	1    3150 2750
@@
 F 0 "R25" H 2870 2896 50  0000 L CNN
 F 1 "5.1 k" H 2870 2805 50  0000 L CNN
-F 2 "" V 2730 2850 50  0001 C CNN
+F 2 "Resistor_SMD:R_0603_1608Metric_Pad1.05x0.95mm_HandSolder" V 2730 2850 50  0001 C CNN
 F 3 "~" H 2800 2850 50  0001 C CNN
 	1    2800 2850
@@
 Wire Wire Line
 	1650 3200 1650 3100
-Connection ~ 1650 3200
 Wire Wire Line
 	1650 3000 1650 2900
@@
 Wire Wire Line
 	2600 4500 4650 4500
-Connection ~ 1650 2900
 Wire Wire Line
 	2500 4400 2500 3200
@@
 Wire Wire Line
 	6350 2150 6650 2150
-$Comp
-L power:PWR_FLAG #FLG0104
-U 1 1 5DD1AB73
-P 1300 1750
-F 0 "#FLG0104" H 1300 1825 50  0001 C CNN
-F 1 "PWR_FLAG" V 1300 1877 50  0000 L CNN
-F 2 "" H 1300 1750 50  0001 C CNN
-F 3 "~" H 1300 1750 50  0001 C CNN
-	1    1300 1750
-	0    -1   -1   0
-$EndComp
 Wire Wire Line
 	6650 5550 6750 5550
@@
 Wire Wire Line
 	2050 2400 3550 2400
+$Comp
+L Snack_Machine:USB_C_Receptacle_USB2.0 J3
+U 1 1 5DBD034E
+P 1050 3000
+F 0 "J3" H 1157 3867 50  0000 C CNN
+F 1 "USB_C_Receptacle_USB2.0" H 1157 3776 50  0000 C CNN
+F 2 "Snack Machine:USB_C_Receptacle_HRO_TYPE-C-31-M-12" H 1200 3000 50  0001 C CNN
+F 3 "https://www.usb.org/sites/default/files/documents/usb_type-c.zip" H 1200 3000 50  0001 C CNN
+	1    1050 3000
+	1    0    0    -1
+$EndComp
+Connection ~ 1650 2900
+Connection ~ 1650 3200
+NoConn ~ 7450 3250
+NoConn ~ 7450 3350
+NoConn ~ 7450 3450
+NoConn ~ 7450 3550
 $EndSCHEMATC

Commit message: Rotated serial ports around to make routing easier
Changed lines of the file:
@@
 	4050 3550 4550 3550
 Connection ~ 4050 3550
-Text Label 4700 3550 0    50   ~ 0
+Text Label 5050 3550 2    50   ~ 0
 USBVCC
 $Comp
@@
 NoConn ~ 7450 3450
 NoConn ~ 7450 3550
+$Comp
+L power:PWR_FLAG #FLG0102
+U 1 1 5DF705E2
+P 6350 2150
+F 0 "#FLG0102" H 6350 2225 50  0001 C CNN
+F 1 "PWR_FLAG" V 6350 2277 50  0000 L CNN
+F 2 "" H 6350 2150 50  0001 C CNN
+F 3 "~" H 6350 2150 50  0001 C CNN
+	1    6350 2150
+	0    -1   -1   0
+$EndComp
 $EndSCHEMATC

Commit message: Sourcing parts
Parts:
- R11: renamed from R25; value 5.1 k -> 5k1; Part Number (none) -> RC0603FR-075K1L
- R25: renamed from R26; value 5.1 k -> 5k1; Part Number (none) -> RC0603FR-075K1L
- Y2: footprint Crystal:Resonator_SMD_muRata_CSTxExxV-3Pin_3.0x1.1mm_HandSoldering -> Snack Machine:Resonator_SMD_ECS-CR2-16.00-B-TR; Manufacturer Murata -> ECS; Part Number CSTCE16M0V53C-R0 -> ECS-CR2-16.00-B-TR
- renumbered C25 to C17, C26 to C18, C27 to C19, C29 to C20, C30 to C23, C23 to C7, C24 to C9, J17 to J13, R55 to R26, R56 to R32, R57 to R33, R58 to R34, R59 to R35, R60 to R36, R61 to R37, R62 to R38, R63 to R39

Commit message: Fixing some small issues here and there
Connections:
- net labels removed: MICRO_RX, MICRO_TX
Changed lines of the file:
@@
 Comment4 ""
 $EndDescr
-Text HLabel 8500 4650 2    50   Input ~ 0
-RX_USB
-Text HLabel 8500 4550 2    50   Input ~ 0
-TX_USB
 $Comp
 L Device:R R32
@@
 Text Label 5550 3550 0    50   ~ 0
 MICRO_D-
-Text Label 7450 4550 0    50   ~ 0
-MICRO_TX
-Text Label 7450 4650 0    50   ~ 0
-MICRO_RX
 Wire Wire Line
 	1650 2400 2050 2400
@@
 	0    -1   -1   0
 $EndComp
+Text HLabel 8500 4650 2    50   Input ~ 0
+TX_USB
+Text HLabel 8500 4550 2    50   Input ~ 0
+RX_USB
 $EndSCHEMATC

Commit message: Added part number, manufacturer, and personal bin numbers
Parts:
- C17, C7: Bin (none) -> 18
- C18: Bin (none) -> 7; Manufacturer TDk -> TDK
- C19, C20: Bin (none) -> 7
- C23, C9: Bin (none) -> 2
- D4: Bin (none) -> 14
- D5, D6: Bin (none) -> 3
- F2: Bin (none) -> 13
- R11, R25: Bin (none) -> 24; Manufacturer (none) -> Yageo
- R26: Bin (none) -> 17
- R32, R33: Bin (none) -> 22
- R34: Bin (none) -> 10
- R35, R36, R37, R38, R39: Bin (none) -> 1
- RV1, RV2: Bin (none) -> 26
- Y2: Bin (none) -> 28
Other:
- note removed: "NOTE: Connect PAD to GND"
Changed lines of the file:
@@
 F 4 "RC0603FR-0722RL" V 5000 4400 50  0001 C CNN "Part Number"
 F 5 "Yageo" V 5000 4400 50  0001 C CNN "Manufacturer"
+F 6 "22" V 5000 4400 50  0001 C CNN "Bin"
 	1    5000 4400
 	0    1    1    0
@@
 F 4 "RC0603FR-0722RL" V 5000 4500 50  0001 C CNN "Part Number"
 F 5 "Yageo" V 5000 4500 50  0001 C CNN "Manufacturer"
+F 6 "22" V 5000 4500 50  0001 C CNN "Bin"
 	1    5000 4500
 	0    1    1    0
@@
 F 4 "RC0603FR-071KL" V 8150 4550 50  0001 C CNN "Part Number"
 F 5 "Yageo" V 8150 4550 50  0001 C CNN "Manufacturer"
+F 6 "1" V 8150 4550 50  0001 C CNN "Bin"
 	1    8150 4550
 	0    1    1    0
@@
 F 4 "RC0603FR-071KL" V 8150 4650 50  0001 C CNN "Part Number"
 F 5 "Yageo" V 8150 4650 50  0001 C CNN "Manufacturer"
+F 6 "1" V 8150 4650 50  0001 C CNN "Bin"
 	1    8150 4650
 	0    1    1    0
@@
 F 4 "150060YS75000" V 9200 4500 50  0001 C CNN "Part Number"
 F 5 "Würth Elektronik" V 9200 4500 50  0001 C CNN "Manufacturer"
+F 6 "3" V 9200 4500 50  0001 C CNN "Bin"
 	1    9200 4500
 	0    -1   -1   0
@@
 F 4 "150060YS75000" V 9550 4500 50  0001 C CNN "Part Number"
 F 5 "Würth Elektronik" V 9550 4500 50  0001 C CNN "Manufacturer"
+F 6 "3" V 9550 4500 50  0001 C CNN "Bin"
 	1    9550 4500
 	0    -1   -1   0
@@
 F 4 "RC0603FR-071KL" H 9200 4100 50  0001 C CNN "Part Number"
 F 5 "Yageo" H 9200 4100 50  0001 C CNN "Manufacturer"
+F 6 "1" H 9200 4100 50  0001 C CNN "Bin"
 	1    9200 4100
 	-1   0    0    1
@@
 F 4 "RC0603FR-071KL" H 9550 4100 50  0001 C CNN "Part Number"
 F 5 "Yageo" H 9550 4100 50  0001 C CNN "Manufacturer"
+F 6 "1" H 9550 4100 50  0001 C CNN "Bin"
 	1    9550 4100
 	-1   0    0    1
@@
 F 4 "RC0603FR-0710KL" H 5800 1150 50  0001 C CNN "Part Number"
 F 5 "Yageo" H 5800 1150 50  0001 C CNN "Manufacturer"
+F 6 "10" H 5800 1150 50  0001 C CNN "Bin"
 	1    5800 1150
 	1    0    0    -1
@@
 F 4 "RC0603FR-071ML" H 4450 2500 50  0001 C CNN "Part Number"
 F 5 "Yageo" H 4450 2500 50  0001 C CNN "Manufacturer"
+F 6 "17" H 4450 2500 50  0001 C CNN "Bin"
 	1    4450 2500
 	1    0    0    -1
@@
 F 4 "C0603C220J1GACTU" H 3950 2900 50  0001 C CNN "Part Number"
 F 5 "KEMET" H 3950 2900 50  0001 C CNN "Manufacturer"
+F 6 "18" H 3950 2900 50  0001 C CNN "Bin"
 	1    3950 2900
 	-1   0    0    1
@@
 F 4 "C0603C220J1GACTU" H 4350 2900 50  0001 C CNN "Part Number"
 F 5 "KEMET" H 4350 2900 50  0001 C CNN "Manufacturer"
+F 6 "18" H 4350 2900 50  0001 C CNN "Bin"
 	1    4350 2900
 	-1   0    0    1
@@
 F 4 "C1608X7R1A105K080AC" H 6750 1150 50  0001 C CNN "Part Number"
 F 5 "TDK" H 6750 1150 50  0001 C CNN "Manufacturer"
+F 6 "7" H 6750 1150 50  0001 C CNN "Bin"
 	1    6750 1150
 	1    0    0    -1
@@
 F 4 "RC0603FR-071KL" H 8150 5300 50  0001 C CNN "Part Number"
 F 5 "Yageo" H 8150 5300 50  0001 C CNN "Manufacturer"
+F 6 "1" H 8150 5300 50  0001 C CNN "Bin"
 	1    8150 5300
 	-1   0    0    1
@@
 F 4 "CC0603KRX7R9BB104" V 8500 5050 50  0001 C CNN "Part Number"
 F 5 "Yageo" V 8500 5050 50  0001 C CNN "Manufacturer"
+F 6 "2" V 8500 5050 50  0001 C CNN "Bin"
 	1    8500 5050
 	0    1    1    0
@@
 F 2 "Resistor_SMD:R_0603_1608Metric_Pad1.05x0.95mm_HandSolder" V 4580 4750 50  0001 C CNN
 F 3 "~" H 4650 4750 50  0001 C CNN
-F 4 "Bourns" H 4650 4750 50  0001 C CNN "Manufacturer"
-F 5 "CG0603MLC-05E" H 4650 4750 50  0001 C CNN "Part Number"
+F 4 "CG0603MLC-05E" H 4650 4750 50  0001 C CNN "Part Number"
+F 5 "Bourns" H 4650 4750 50  0001 C CNN "Manufacturer"
+F 6 "26" H 4650 4750 50  0001 C CNN "Bin"
 	1    4650 4750
 	1    0    0    -1
@@
 F 2 "Resistor_SMD:R_0603_1608Metric_Pad1.05x0.95mm_HandSolder" V 3880 4750 50  0001 C CNN
 F 3 "~" H 3950 4750 50  0001 C CNN
-F 4 "Bourns" H 3950 4750 50  0001 C CNN "Manufacturer"
-F 5 "CG0603MLC-05E" H 3950 4750 50  0001 C CNN "Part Number"
+F 4 "CG0603MLC-05E" H 3950 4750 50  0001 C CNN "Part Number"
+F 5 "Bourns" H 3950 4750 50  0001 C CNN "Manufacturer"
+F 6 "26" H 3950 4750 50  0001 C CNN "Bin"
 	1    3950 4750
 	1    0    0    -1
@@
 F 2 "Snack Machine:MF-MSMF050-2" H 3850 3350 50  0001 L CNN
 F 3 "~" H 3800 3550 50  0001 C CNN
-F 4 "Bourns" V 3800 3550 50  0001 C CNN "Manufacturer"
-F 5 "MF-MSMF050-2" V 3800 3550 50  0001 C CNN "Part Number"
+F 4 "MF-MSMF050-2" V 3800 3550 50  0001 C CNN "Part Number"
+F 5 "Bourns" V 3800 3550 50  0001 C CNN "Manufacturer"
+F 6 "13" V 3800 3550 50  0001 C CNN "Bin"
 	1    3800 3550
 	0    1    1    0
@@
 F 4 "CC0603KRX7R9BB104" H 4050 3800 50  0001 C CNN "Part Number"
 F 5 "Yageo" H 4050 3800 50  0001 C CNN "Manufacturer"
+F 6 "2" H 4050 3800 50  0001 C CNN "Bin"
 	1    4050 3800
 	1    0    0    -1
@@
 F 3 "~" H 4550 3800 50  0001 C CNN
 F 4 "C1608X7R1A105K080AC" H 4550 3800 50  0001 C CNN "Part Number"
-F 5 "TDk" H 4550 3800 50  0001 C CNN "Manufacturer"
+F 5 "TDK" H 4550 3800 50  0001 C CNN "Manufacturer"
+F 6 "7" H 4550 3800 50  0001 C CNN "Bin"
 	1    4550 3800
 	1    0    0    -1
@@
 F 4 "C1608X7R1A105K080AC" H 5750 4000 50  0001 C CNN "Part Number"
 F 5 "TDK" H 5750 4000 50  0001 C CNN "Manufacturer"
+F 6 "7" H 5750 4000 50  0001 C CNN "Bin"
 	1    5750 4000
 	1    0    0    -1
@@
 Wire Wire Line
 	5750 3750 6050 3750
-Text Notes 6200 5950 0    50   ~ 0
-NOTE: Connect PAD to GND
 $Comp
 L Device:D D4
@@
 F 4 "Bourns" V 6100 1150 50  0001 C CNN "Manufacturer"
 F 5 "CD1206-S01575" V 6100 1150 50  0001 C CNN "Part Number"
+F 6 "14" V 6100 1150 50  0001 C CNN "Bin"
 	1    6100 1150
 	0    1    1    0
@@
 F 4 "ECS" H 5100 2500 50  0001 C CNN "Manufacturer"
 F 5 "ECS-CR2-16.00-B-TR" H 5100 2500 50  0001 C CNN "Part Number"
+F 6 "28" V 5100 2500 50  0001 C CNN "Bin"
 	1    5100 2500
 	0    1    -1   0
@@
 F 3 "~" H 3150 2750 50  0001 C CNN
 F 4 "RC0603FR-075K1L" H 3150 2750 50  0001 C CNN "Part Number"
+F 5 "Yageo" H 3150 2750 50  0001 C CNN "Manufacturer"
+F 6 "24" H 3150 2750 50  0001 C CNN "Bin"
 	1    3150 2750
 	1    0    0    -1
@@
 F 3 "~" H 2800 2850 50  0001 C CNN
 F 4 "RC0603FR-075K1L" H 2800 2850 50  0001 C CNN "Part Number"
+F 5 "Yageo" H 2800 2850 50  0001 C CNN "Manufacturer"
+F 6 "24" H 2800 2850 50  0001 C CNN "Bin"
 	1    2800 2850
 	1    0    0    -1

Commit message: Improving some grounding issues
Connections:
- wire segments 92 -> 95
- no-connect marks 15 -> 12
Changed lines of the file:
@@
 	8500 4650 8300 4650
 NoConn ~ 7450 3850
-NoConn ~ 7450 3750
-NoConn ~ 7450 4350
 $Comp
 L Device:LED D5
@@
 NoConn ~ 7450 4050
 NoConn ~ 7450 4150
-NoConn ~ 7450 4450
 NoConn ~ 7450 4950
 Text Notes 9900 5300 2    50   ~ 0
@@
 Text HLabel 8500 4550 2    50   Input ~ 0
 RX_USB
+Wire Wire Line
+	7450 3750 7550 3750
+Wire Wire Line
+	7450 4350 7550 4350
+Wire Wire Line
+	7450 4450 7550 4450
+$Comp
+L power:GND #PWR?
+U 1 1 5E906C18
+P 7550 3750
+F 0 "#PWR?" H 7550 3500 50  0001 C CNN
+F 1 "GND" V 7555 3622 50  0000 R CNN
+F 2 "" H 7550 3750 50  0001 C CNN
+F 3 "" H 7550 3750 50  0001 C CNN
+	1    7550 3750
+	0    -1   -1   0
+$EndComp
+$Comp
+L power:GND #PWR?
+U 1 1 5E90759A
+P 7550 4350
+F 0 "#PWR?" H 7550 4100 50  0001 C CNN
+F 1 "GND" V 7555 4222 50  0000 R CNN
+F 2 "" H 7550 4350 50  0001 C CNN
+F 3 "" H 7550 4350 50  0001 C CNN
+	1    7550 4350
+	0    -1   -1   0
+$EndComp
+$Comp
+L power:GND #PWR?
+U 1 1 5E907ADA
+P 7550 4450
+F 0 "#PWR?" H 7550 4200 50  0001 C CNN
+F 1 "GND" V 7555 4322 50  0000 R CNN
+F 2 "" H 7550 4450 50  0001 C CNN
+F 3 "" H 7550 4450 50  0001 C CNN
+	1    7550 4450
+	0    -1   -1   0
+$EndComp
 $EndSCHEMATC

Commit message: Committing changes to the circuit board
Parts:
- J3: Bin (none) -> 37, 38, 39; Manufacturer (none) -> JAE Electronics; Part Number (none) -> DX07S016JA1R1500
Changed lines of the file:
@@
 F 2 "Snack Machine:USB_C_Receptacle_HRO_TYPE-C-31-M-12" H 1200 3000 50  0001 C CNN
 F 3 "https://www.usb.org/sites/default/files/documents/usb_type-c.zip" H 1200 3000 50  0001 C CNN
+F 4 "37, 38, 39" H 1050 3000 50  0001 C CNN "Bin"
+F 5 "JAE Electronics" H 1050 3000 50  0001 C CNN "Manufacturer"
+F 6 "DX07S016JA1R1500" H 1050 3000 50  0001 C CNN "Part Number"
 	1    1050 3000
 	1    0    0    -1
@@
 	7450 4450 7550 4450
 $Comp
-L power:GND #PWR?
+L power:GND #PWR0115
 U 1 1 5E906C18
 P 7550 3750
-F 0 "#PWR?" H 7550 3500 50  0001 C CNN
+F 0 "#PWR0115" H 7550 3500 50  0001 C CNN
 F 1 "GND" V 7555 3622 50  0000 R CNN
 F 2 "" H 7550 3750 50  0001 C CNN
@@
 $EndComp
 $Comp
-L power:GND #PWR?
+L power:GND #PWR0116
 U 1 1 5E90759A
 P 7550 4350
-F 0 "#PWR?" H 7550 4100 50  0001 C CNN
+F 0 "#PWR0116" H 7550 4100 50  0001 C CNN
 F 1 "GND" V 7555 4222 50  0000 R CNN
 F 2 "" H 7550 4350 50  0001 C CNN
@@
 $EndComp
 $Comp
-L power:GND #PWR?
+L power:GND #PWR0117
 U 1 1 5E907ADA
 P 7550 4450
-F 0 "#PWR?" H 7550 4200 50  0001 C CNN
+F 0 "#PWR0117" H 7550 4200 50  0001 C CNN
 F 1 "GND" V 7555 4322 50  0000 R CNN
 F 2 "" H 7550 4450 50  0001 C CNN
